Commit message: [适配] 适配ros，第一次提交代码，可以实现基本运动

File: rokae/rokae_description/urdf/xMateCR7.urdf.xacro (robot description, xacro)
@@ -39,5 +39,5 @@
     <parent link="${nameofManipulator}_base"/>
     <child link="${nameofManipulator}_link1"/>
- <limit effort="300" lower="-3.1416" upper="3.1416" velocity="10"/>
+ <limit effort="300" lower="-3.054" upper="3.054" velocity="8"/>
     <axis xyz="0 0 1"/>
     <origin rpy="0 0 0" xyz="0 0 0"/>
@@ -45,9 +45,9 @@
 <transmission name="tran1">
     <type>transmission_interface/SimpleTransmission</type>
-    <joint name="xmate_joint_1">
-      <hardwareInterface>EffortJointInterface</hardwareInterface>
+    <joint name="joint1">
+      <hardwareInterface>PositionJointInterface</hardwareInterface>
     </joint>
     <actuator name="motor1">
-      <hardwareInterface>EffortJointInterface</hardwareInterface>
+      <hardwareInterface>PositionJointInterface</hardwareInterface>
       <mechanicalReduction>1</mechanicalReduction>
     </actuator>
@@ -77,5 +77,5 @@
     <parent link="${nameofManipulator}_link1"/>
     <child link="${nameofManipulator}_link2"/>
-  <limit effort="300" lower="-3.1416" upper="3.1416" velocity="10"/>
+  <limit effort="300" lower="-3.054" upper="3.054" velocity="8"/>
     <axis xyz="0 1 0"/>
 	<origin rpy="0 0 0" xyz="0 0 0.296"/>
@@ -83,9 +83,9 @@
    <transmission name="tran2">
      <type>transmission_interface/SimpleTransmission</type>
-    <joint name="xmate_joint_2">
-      <hardwareInterface>EffortJointInterface</hardwareInterface>
+    <joint name="joint2">
+      <hardwareInterface>PositionJointInterface</hardwareInterface>
     </joint>
     <actuator name="motor2">
-      <hardwareInterface>EffortJointInterface</hardwareInterface>
+      <hardwareInterface>PositionJointInterface</hardwareInterface>
       <mechanicalReduction>1</mechanicalReduction>
     </actuator>
@@ -115,5 +115,5 @@
     <parent link="${nameofManipulator}_link2"/>
     <child link="${nameofManipulator}_link3"/>
-  <limit effort="300" lower="-4.9742" upper="4.9742" velocity="10"/>
+  <limit effort="300" lower="-3.054" upper="3.054" velocity="8"/>
     <axis xyz="0 -1 0"/>
     <origin rpy="0 0 0" xyz="0 0 0.49"/>
@@ -121,9 +121,9 @@
    <transmission name="tran3">
     <type>transmission_interface/SimpleTransmission</type>
-    <joint name="xmate_joint_3">
-      <hardwareInterface>EffortJointInterface</hardwareInterface>
+    <joint name="joint3">
+      <hardwareInterface>PositionJointInterface</hardwareInterface>
     </joint>
     <actuator name="motor3">
-      <hardwareInterface>EffortJointInterface</hardwareInterface>
+      <hardwareInterface>PositionJointInterface</hardwareInterface>
       <mechanicalReduction>1</mechanicalReduction>
     </actuator>
@@ -153,5 +153,5 @@
     <parent link="${nameofManipulator}_link3"/>
     <child link="${nameofManipulator}_link4"/>
-   <limit effort="300" lower="-3.1416" upper="3.1416" velocity="10"/>
+   <limit effort="300" lower="-3.054" upper="3.054" velocity="8"/>
 <!--     lower="-2.79" upper="2.79" -->
     <axis xyz="0 0 1"/>
@@ -161,9 +161,9 @@
   <transmission name="tran4">
     <type>transmission_interface/SimpleTransmission</type>
-    <joint name="xmate_joint_4">
-      <hardwareInterface>EffortJointInterface</hardwareInterface>
+    <joint name="joint4">
+      <hardwareInterface>PositionJointInterface</hardwareInterface>
     </joint>
     <actuator name="motor4">
-      <hardwareInterface>EffortJointInterface</hardwareInterface>
+      <hardwareInterface>PositionJointInterface</hardwareInterface>
       <mechanicalReduction>1</mechanicalReduction>
     </actuator>
@@ -193,5 +193,5 @@
     <parent link="${nameofManipulator}_link4"/>
     <child link="${nameofManipulator}_link5"/>
-  <limit effort="300" lower="-3.1416" upper="3.1416" velocity="10"/>
+  <limit effort="300" lower="-3.054" upper="3.054" velocity="8"/>
     <axis xyz="0 -1 0"/>
    <origin rpy="0 0 0" xyz="0 -0.151 0"/>
@@ -199,9 +199,9 @@
   <transmission name="tran5">
     <type>transmission_interface/SimpleTransmission</type>
-    <joint name="xmate_joint_5">
-      <hardwareInterface>EffortJointInterface</hardwareInterface>
+    <joint name="joint5">
+      <hardwareInterface>PositionJointInterface</hardwareInterface>
     </joint>
     <actuator name="motor5">
-      <hardwareInterface>EffortJointInterface</hardwareInterface>
+      <hardwareInterface>PositionJointInterface</hardwareInterface>
       <mechanicalReduction>1</mechanicalReduction>
     </actuator>
@@ -231,5 +231,5 @@
     <parent link="${nameofManipulator}_link5"/>
     <child link="${nameofManipulator}_link6"/>
-   <limit effort="300" lower="-6.1082" upper="6.1082" velocity="10"/>
+   <limit effort="300" lower="-3.054" upper="3.054" velocity="8"/>
     <axis xyz="0 0 1"/>
     <origin rpy="0.0 0.0 0" xyz="0 0 0.1265" />
@@ -237,9 +237,9 @@
   <transmission name="tran6">
     <type>transmission_interface/SimpleTransmission</type>
-    <joint name="xmate_joint_6">
-      <hardwareInterface>EffortJointInterface</hardwareInterface>
+    <joint name="joint6">
+      <hardwareInterface>PositionJointInterface</hardwareInterface>
     </joint>
     <actuator name="motor6">
-      <hardwareInterface>EffortJointInterface</hardwareInterface>
+      <hardwareInterface>PositionJointInterface</hardwareInterface>
       <mechanicalReduction>1</mechanicalReduction>
     </actuator>
