Commit message: rokae_driver编写 修正一些moveit_config包

File: rokae/rokae_description/urdf/xMateER7.ros2_control.xacro (robot description, xacro)
@@ -24,30 +24,30 @@
         </xacro:unless>
       </hardware>
-      <joint name="joint1">
+      <joint name="xMate7_joint_1">
         <command_interface name="position"/>
         <state_interface name="position"/>
         <state_interface name="velocity"/>
       </joint>
-      <joint name="joint2">
+      <joint name="xMate7_joint_2">
         <command_interface name="position"/>
         <state_interface name="position"/>
         <state_interface name="velocity"/>
       </joint>
-      <joint name="joint3">
+      <joint name="xMate7_joint_3">
         <command_interface name="position"/>
         <state_interface name="position"/>
         <state_interface name="velocity"/>
       </joint>
-      <joint name="joint4">
+      <joint name="xMate7_joint_4">
         <command_interface name="position"/>
         <state_interface name="position"/>
         <state_interface name="velocity"/>
       </joint>
-      <joint name="joint5">
+      <joint name="xMate7_joint_5">
         <command_interface name="position"/>
         <state_interface name="position"/>
         <state_interface name="velocity"/>
       </joint>
-      <joint name="joint6">
+      <joint name="xMate7_joint_6">
         <command_interface name="position"/>
         <state_interface name="position"/>

File: rokae/rokae_description/urdf/xMateER7.urdf.xacro (robot description, xacro)
@@ -1,391 +1,285 @@
-<robot
-  name="XME7">
-  <link
-    name="base_link">
-    <inertial>
-      <origin
-        xyz="0.0218436668217748 0.0163699016708871 0.0336311683087049"
-        rpy="0 0 0" />
-      <mass
-        value="5.27506583792117" />
-      <inertia
-        ixx="0"
-        ixy="0"
-        ixz="0"
-        iyy="0"
-        iyz="0"
-        izz="0" />
-    </inertial>
-    <visual>
-      <origin
-        xyz="0 0 0"
-        rpy="0 0 0" />
-      <geometry>
-        <mesh
-          filename="package://XME7/meshes/base_link.STL" />
-      </geometry>
-      <material
-        name="">
-        <color
-          rgba="0.592156862745098 0.666666666666667 0.682352941176471 1" />
-      </material>
-    </visual>
-    <collision>
-      <origin
-        xyz="0 0 0"
-        rpy="0 0 0" />
-      <geometry>
-        <mesh
-          filename="package://XME7/meshes/base_link.STL" />
-      </geometry>
-    </collision>
-  </link>
-  <link
-    name="link1">
-    <inertial>
-      <origin
-        xyz="5.79402105674309E-06 -0.0307935710783682 0.141714967811122"
-        rpy="0 0 0" />
-      <mass
-        value="3.69864967968703" />
-      <inertia
-        ixx="0.0292381087544826"
-        ixy="0"
-        ixz="0"
-        iyy="0.0462803078466669"
-        iyz="0"
-        izz="0.024610077994494" />
-    </inertial>
-    <visual>
-      <origin
-        xyz="0 0 0"
-        rpy="0 0 0" />
-      <geometry>
-        <mesh
-          filename="package://XME7/meshes/link1.STL" />
-      </geometry>
-      <material
-        name="">
-        <color
-          rgba="0.592156862745098 0.666666666666667 0.682352941176471 1" />
-      </material>
-    </visual>
-    <collision>
-      <origin
-        xyz="0 0 0"
-        rpy="0 0 0" />
-      <geometry>
-        <mesh
-          filename="package://XME7/meshes/link1.STL" />
-      </geometry>
-    </collision>
-  </link>
-  <joint
-    name="joint1"
-    type="revolute">
-    <origin
-      xyz="0.040901 -0.033668 0.13818"
-      rpy="-2.8368E-15 0 -3.14" />
-    <parent
-      link="base_link" />
-    <child
-      link="link1" />
-    <axis
-      xyz="0 0 1" />
-    <limit
-      lower="-2.9671"
-      upper="2.9671"
-      effort="0"
-      velocity="0" />
-  </joint>
-  <link
-    name="link2">
-    <inertial>
-      <origin
-        xyz="4.23738311908922E-06 0.200065991468864 -0.0155752111863818"
-        rpy="0 0 0" />
-      <mass
-        value="4.95201979538989" />
-      <inertia
-        ixx="0.0292381087544826"
-        ixy="0"
-        ixz="0"
-        iyy="0.0462803078466669"
-        iyz="0"
-        izz="0.024610077994494" />
-    </inertial>
-    <visual>
-      <origin
-        xyz="0 0 0"
-        rpy="0 0 0" />
-      <geometry>
-        <mesh
-          filename="package://XME7/meshes/link2.STL" />
-      </geometry>
-      <material
-        name="">
-        <color
-          rgba="0.592156862745098 0.666666666666667 0.682352941176471 1" />
-      </material>
-    </visual>
-    <collision>
-      <origin
-        xyz="0 0 0"
-        rpy="0 0 0" />
-      <geometry>
-        <mesh
-          filename="package://XME7/meshes/link2.STL" />
-      </geometry>
-    </collision>
-  </link>
-  <joint
-    name="joint2"
-    type="revolute">
-    <origin
-      xyz="0 0 0.207999999952273"
-      rpy="1.5707963267949 0 0" />
-    <parent
-      link="link1" />
-    <child
-      link="link2" />
-    <axis
-      xyz="0 0 0.99999999999966" />
-    <limit
-      lower="-2.0943951023932"
-      upper="2.0943951023932"
-      effort="0"
-      velocity="0" />
-  </joint>
-  <link
-    name="link3">
-    <inertial>
-      <origin
-        xyz="3.25348652711194E-06 0.0327880429508358 0.0757964191760764"
-        rpy="0 0 0" />
-      <mass
-        value="1.79724502165651" />
-      <inertia
-        ixx="0.0292381087544826"
-        ixy="0"
-        ixz="0"
-        iyy="0.0462803078466669"
-        iyz="0"
-        izz="0.024610077994494" />
-    </inertial>
-    <visual>
-      <origin
-        xyz="0 0 0"
-        rpy="0 0 0" />
-      <geometry>
-        <mesh
-          filename="package://XME7/meshes/link3.STL" />
-      </geometry>
-      <material
-        name="">
-        <color
-          rgba="0.592156862745098 0.666666666666667 0.682352941176471 1" />
-      </material>
-    </visual>
-    <collision>
-      <origin
-        xyz="0 0 0"
-        rpy="0 0 0" />
-      <geometry>
-        <mesh
-          filename="package://XME7/meshes/link3.STL" />
-      </geometry>
-    </collision>
-  </link>
-  <joint
-    name="joint3"
-    type="revolute">
-    <origin
-      xyz="0 0.437499909676678 0"
-      rpy="-1.57079759282358 0 0" />
-    <parent
-      link="link2" />
-    <child
-      link="link3" />
-    <axis
-      xyz="0 -0.999999999998858 0" />
-    <limit
-      lower="-2.0943951023932"
-      upper="2.0943951023932"
-      effort="0"
-      velocity="0" />
-  </joint>
-  <link
-    name="link4">
-    <inertial>
-      <origin
-        xyz="9.69897826796212E-06 -0.0230961404656154 0.13591016450192"
-        rpy="0 0 0" />
-      <mass
-        value="1.71426245435884" />
-      <inertia
-        ixx="0.0292381087544826"
-        ixy="0"
-        ixz="0"
-        iyy="0.0462803078466669"
-        iyz="0"
-        izz="0.024610077994494" />
-    </inertial>
-    <visual>
-      <origin
-        xyz="0 0 0"
-        rpy="0 0 0" />
-      <geometry>
-        <mesh
-          filename="package://XME7/meshes/link4.STL" />
-      </geometry>
-      <material
-        name="">
-        <color
-          rgba="0.592156862745098 0.666666666666667 0.682352941176471 1" />
-      </material>
-    </visual>
-    <collision>
-      <origin
-        xyz="0 0 0"
-        rpy="0 0 0" />
-      <geometry>
-        <mesh
-          filename="package://XME7/meshes/link4.STL" />
-      </geometry>
-    </collision>
-  </link>
-  <joint
-    name="joint4"
-    type="revolute">
-    <origin
-      xyz="0 0 0.20999999662933"
-      rpy="0 0 0" />
-    <parent
-      link="link3" />
-    <child
-      link="link4" />
-    <axis
-      xyz="0 0 0.999999999998397" />
-    <limit
-      lower="-2.96705972839037"
-      upper="2.96705972839037"
-      effort="0"
-      velocity="0" />
-  </joint>
-  <link
-    name="link5">
-    <inertial>
-      <origin
-        xyz="1.67277909225855E-05 0.0189580631840378 0.0947781921805828"
-        rpy="0 0 0" />
-      <mass
-        value="1.29891490887537" />
-      <inertia
-        ixx="0.0292381087544826"
-        ixy="0"
-        ixz="0"
-        iyy="0.0462803078466669"
-        iyz="0"
-        izz="0.024610077994494" />
-    </inertial>
-    <visual>
-      <origin
-        xyz="0 0 0"
-        rpy="0 0 0" />
-      <geometry>
-        <mesh
-          filename="package://XME7/meshes/link5.STL" />
-      </geometry>
-      <material
-        name="">
-        <color
-          rgba="0.592156862745098 0.666666666666667 0.682352941176471 1" />
-      </material>
-    </visual>
-    <collision>
-      <origin
-        xyz="0 0 0"
-        rpy="0 0 0" />
-      <geometry>
-        <mesh
-          filename="package://XME7/meshes/link5.STL" />
-      </geometry>
-    </collision>
-  </link>
-  <joint
-    name="joint5"
-    type="revolute">
-    <origin
-      xyz="0 0 0.202499820575684"
-      rpy="0 0 0" />
-    <parent
-      link="link4" />
-    <child
-      link="link5" />
-    <axis
-      xyz="0 -0.999999999998397 0" />
-    <limit
-      lower="-2.0943951023932"
-      upper="2.0943951023932"
-      effort="0"
-      velocity="0" />
-  </joint>
-  <link
-    name="link6">
-    <inertial>
-      <origin
-        xyz="4.41762519806932E-05 0.0209443148419796 0.0816293943338553"
-        rpy="0 0 0" />
-      <mass
-        value="0.597615641843439" />
-      <inertia
-        ixx="0.0292381087544826"
-        ixy="0"
-        ixz="0"
-        iyy="0.0462803078466669"
-        iyz="0"
-        izz="0.024610077994494" />
-    </inertial>
-    <visual>
-      <origin
-        xyz="0 0 0"
-        rpy="0 0 0" />
-      <geometry>
-        <mesh
-          filename="package://XME7/meshes/link6.STL" />
-      </geometry>
-      <material
-        name="">
-        <color
-          rgba="0.592156862745098 0.666666666666667 0.682352941176471 1" />
-      </material>
-    </visual>
-    <collision>
-      <origin
-        xyz="0 0 0"
-        rpy="0 0 0" />
-      <geometry>
-        <mesh
-          filename="package://XME7/meshes/link6.STL" />
-      </geometry>
-    </collision>
-  </link>
-  <joint
-    name="joint6"
-    type="revolute">
-    <origin
-      xyz="0 0 0.147077572634105"
-      rpy="0 0 0" />
-    <parent
-      link="link5" />
-    <child
-      link="link6" />
-    <axis
-      xyz="0 0 0.999999999998397" />
-    <limit
-      lower="-3.1415926535898"
-      upper="3.1415926535898"
-      effort="0"
-      velocity="0" />
-  </joint>
+<?xml version='1.0' encoding='UTF-8'?>
+<robot xmlns:xacro="http://www.ros.org/wiki/xacro" name="xMate7">
+  <!-- Constants for robot dimensions -->
+  <!-- <material name="black">
+    <color rgba="0.0 0.0 0.0 1.0"/>
+  </material>
+  <material name="blue">
+    <color rgba="0.0 0.0 0.8 1.0"/>
+  </material>
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