Commit message: 第二版，硬件接口实例化，六轴七轴HMI测试通过

File: rokae/rokae_description/urdf/xMate.urdf.xacro (robot description, xacro)
@@ -1,17 +1,32 @@
-<?xml version="1.0" encoding="utf-8"?>
-<robot xmlns:xacro="http://www.ros.org/wiki/xacro" name="xMate">
-  <!-- 'xMate_type' values: xMate_CR7 -->
-  <xacro:arg name="xMate_type" default="xMate_CR7"/>
-  <!-- import main macro -->
+<?xml version="1.0"?>
+<robot xmlns:xacro="http://www.ros.org/wiki/xacro" name="xMate_robot">
+  <!-- 启动参数（launch.py 会传 robot_type） -->
+  <xacro:arg name="robot_type" default="CR7"/>  <!-- 可选: CR7, SR4, ER7p, ER7 -->
+  <xacro:arg name="robot_ip" default="192.168.21.10"/>
+  <xacro:arg name="local_ip" default="192.168.21.131"/>
+  <xacro:arg name="use_fake_hardware" default="false"/>
+  <!-- 引入宏文件 -->
   <xacro:include filename="$(find rokae_description)/urdf/xMate_macro.xacro"/>
-  <!-- parameters -->
-  <xacro:arg name="use_fake_hardware" default="false" />
-  <xacro:arg name="robot_ip" default="192.168.21.10" />
-  <xacro:arg name="local_ip" default="192.168.21.131" />
+  <!-- 先把 launch 传入的 robot_type 映射为可用于表达式的 property -->
+  <xacro:property name="robot_type_prop" value="$(arg robot_type)"/>
+  <!-- 映射出 xMate_type（默认 CR7，再按条件覆盖） -->
+  <xacro:property name="xMate_type" value="xMateCR7"/>
+  <xacro:if value="${robot_type_prop == 'SR4'}">
+    <xacro:property name="xMate_type" value="xMateSR4"/>
+  </xacro:if>
+  <xacro:if value="${robot_type_prop == 'Pro3'}">
+    <xacro:property name="xMate_type" value="xMatePro3"/>
+  </xacro:if>
+  <xacro:if value="${robot_type_prop == 'Pro7'}">
+    <xacro:property name="xMate_type" value="xMatePro7"/>
+  </xacro:if>
+  <xacro:if value="${robot_type_prop == 'ER7'}">
+    <xacro:property name="xMate_type" value="xMateER7"/>
+  </xacro:if>
+  <!-- 调用总宏（只传 xMate_type，内部再按机型 include/调用具体实现） -->
   <xacro:rokae_robot
-    xMate_type="$(arg xMate_type)"
-    robot_ip="$(arg robot_ip)"
-    local_ip="$(arg local_ip)"
-    use_fake_hardware="$(arg use_fake_hardware)">
-  </xacro:rokae_robot>
+      xMate_type="${xMate_type}"
+      robot_ip="$(arg robot_ip)"
+      local_ip="$(arg local_ip)"
+      use_fake_hardware="$(arg use_fake_hardware)"/>
 </robot>

File: rokae/rokae_description/urdf/xMate_macro.xacro (robot description, xacro)
@@ -1,19 +1,61 @@
 <?xml version="1.0"?>
-<robot xmlns:xacro="http://wiki.ros.org/xacro">
+<robot xmlns:xacro="http://www.ros.org/wiki/xacro">
+  <!-- 总宏：根据 xMate_type 选择不同 urdf 与 ros2_control -->
   <xacro:macro name="rokae_robot"
     params="
-    xMate_type
-    robot_ip
-    local_ip
-    use_fake_hardware:=false
-    ">
-    <!-- Rizon 4 or 4s-->
-    <xacro:include filename="$(find rokae_description)/urdf/xMateCR7.urdf.xacro" />
-    <xacro:include filename="$(find rokae_description)/urdf/cr7.ros2_controll.xacro" />
-    <xacro:cr7_ros2_controll
-      use_fake_hardware="${use_fake_hardware}"
-      robot_ip="$(arg robot_ip)"
-      local_ip="$(arg local_ip)"
-    />
+      xMate_type
+      robot_ip
+      local_ip
+      use_fake_hardware:=false">
+    <!-- CR7 -->
+    <xacro:if value="${xMate_type == 'xMateCR7'}">
+      <xacro:include filename="$(find rokae_description)/urdf/xMateCR7.urdf.xacro"/>
+      <xacro:include filename="$(find rokae_description)/urdf/xMateCR7.ros2_controll.xacro"/>
+      <xacro:cr7_ros2_controll
+        robot_ip="${robot_ip}"
+        local_ip="${local_ip}"
+        use_fake_hardware="${use_fake_hardware}"/>
+    </xacro:if>
+    <!-- SR4 -->
+    <xacro:if value="${xMate_type == 'xMateSR4'}">
+      <xacro:include filename="$(find rokae_description)/urdf/xMateSR4.urdf.xacro"/>
+      <xacro:include filename="$(find rokae_description)/urdf/xMateSR4.ros2_controll.xacro"/>
+      <xacro:sr4_ros2_controll
+        robot_ip="${robot_ip}"
+        local_ip="${local_ip}"
+        use_fake_hardware="${use_fake_hardware}"/>
+    </xacro:if>
+    <!-- ER7 -->
+    <xacro:if value="${xMate_type == 'xMateER7'}">
+      <xacro:include filename="$(find rokae_description)/urdf/xMateER7.urdf.xacro"/>
+      <xacro:include filename="$(find rokae_description)/urdf/xMateER7.ros2_controll.xacro"/>
+      <xacro:er7_ros2_controll
+        robot_ip="${robot_ip}"
+        local_ip="${local_ip}"
+        use_fake_hardware="${use_fake_hardware}"/>
+    </xacro:if>
+    <!-- ER7Pro -->
+    <xacro:if value="${xMate_type == 'xMatePro7'}">
+      <xacro:include filename="$(find rokae_description)/urdf/xMatePro7.urdf.xacro"/>
+      <xacro:include filename="$(find rokae_description)/urdf/xMatePro7.ros2_controll.xacro"/>
+      <xacro:er7p_ros2_controll
+        robot_ip="${robot_ip}"
+        local_ip="${local_ip}"
+        use_fake_hardware="${use_fake_hardware}"/>
+    </xacro:if>
+    <!-- ER3Pro -->
+    <xacro:if value="${xMate_type == 'xMatePro3'}">
+      <xacro:include filename="$(find rokae_description)/urdf/xMatePro3.urdf.xacro"/>
+      <xacro:include filename="$(find rokae_description)/urdf/xMatePro3.ros2_controll.xacro"/>
+      <xacro:er3p_ros2_controll
+        robot_ip="${robot_ip}"
+        local_ip="${local_ip}"
+        use_fake_hardware="${use_fake_hardware}"/>
+    </xacro:if>
+    <!-- 其他机型（如有）按同样模式继续加 -->
+    <!--
+    <xacro:if value="${xMate_type == 'xMateER7p'}"> … </xacro:if>
+    <xacro:if value="${xMate_type == 'xMateER7'}"> … </xacro:if>
+    -->
   </xacro:macro>
 </robot>

Commit message: 适配AR5机型，通过use_fake_hardware测试

File: rokae/rokae_description/urdf/xMate.urdf.xacro (robot description, xacro)
@@ -24,4 +24,10 @@
     <xacro:property name="xMate_type" value="xMateER7"/>
   </xacro:if>
+  <xacro:if value="${robot_type_prop == 'AR5L'}">
+    <xacro:property name="xMate_type" value="AR5L"/>
+  </xacro:if>
+  <xacro:if value="${robot_type_prop == 'AR5R'}">
+    <xacro:property name="xMate_type" value="AR5R"/>
+  </xacro:if>
   <!-- 调用总宏（只传 xMate_type，内部再按机型 include/调用具体实现） -->
   <xacro:rokae_robot

File: rokae/rokae_description/urdf/xMate_macro.xacro (robot description, xacro)
@@ -11,6 +11,6 @@
     <xacro:if value="${xMate_type == 'xMateCR7'}">
       <xacro:include filename="$(find rokae_description)/urdf/xMateCR7.urdf.xacro"/>
-      <xacro:include filename="$(find rokae_description)/urdf/xMateCR7.ros2_controll.xacro"/>
-      <xacro:cr7_ros2_controll
+      <xacro:include filename="$(find rokae_description)/urdf/xMateCR7.ros2_control.xacro"/>
+      <xacro:cr7_ros2_control
         robot_ip="${robot_ip}"
         local_ip="${local_ip}"
@@ -20,6 +20,6 @@
     <xacro:if value="${xMate_type == 'xMateSR4'}">
       <xacro:include filename="$(find rokae_description)/urdf/xMateSR4.urdf.xacro"/>
-      <xacro:include filename="$(find rokae_description)/urdf/xMateSR4.ros2_controll.xacro"/>
-      <xacro:sr4_ros2_controll
+      <xacro:include filename="$(find rokae_description)/urdf/xMateSR4.ros2_control.xacro"/>
+      <xacro:sr4_ros2_control
         robot_ip="${robot_ip}"
         local_ip="${local_ip}"
@@ -29,6 +29,6 @@
     <xacro:if value="${xMate_type == 'xMateER7'}">
       <xacro:include filename="$(find rokae_description)/urdf/xMateER7.urdf.xacro"/>
-      <xacro:include filename="$(find rokae_description)/urdf/xMateER7.ros2_controll.xacro"/>
-      <xacro:er7_ros2_controll
+      <xacro:include filename="$(find rokae_description)/urdf/xMateER7.ros2_control.xacro"/>
+      <xacro:er7_ros2_control
         robot_ip="${robot_ip}"
         local_ip="${local_ip}"
@@ -38,6 +38,6 @@
     <xacro:if value="${xMate_type == 'xMatePro7'}">
       <xacro:include filename="$(find rokae_description)/urdf/xMatePro7.urdf.xacro"/>
-      <xacro:include filename="$(find rokae_description)/urdf/xMatePro7.ros2_controll.xacro"/>
-      <xacro:er7p_ros2_controll
+      <xacro:include filename="$(find rokae_description)/urdf/xMatePro7.ros2_control.xacro"/>
+      <xacro:er7p_ros2_control
         robot_ip="${robot_ip}"
         local_ip="${local_ip}"
@@ -47,6 +47,6 @@
     <xacro:if value="${xMate_type == 'xMatePro3'}">
       <xacro:include filename="$(find rokae_description)/urdf/xMatePro3.urdf.xacro"/>
-      <xacro:include filename="$(find rokae_description)/urdf/xMatePro3.ros2_controll.xacro"/>
-      <xacro:er3p_ros2_controll
+      <xacro:include filename="$(find rokae_description)/urdf/xMatePro3.ros2_control.xacro"/>
+      <xacro:er3p_ros2_control
         robot_ip="${robot_ip}"
         local_ip="${local_ip}"
@@ -54,8 +54,22 @@
     </xacro:if>
     <!-- 其他机型（如有）按同样模式继续加 -->
-    <!--
-    <xacro:if value="${xMate_type == 'xMateER7p'}"> … </xacro:if>
-    <xacro:if value="${xMate_type == 'xMateER7'}"> … </xacro:if>
-    -->
+    <!-- AR5L -->
+    <xacro:if value="${xMate_type == 'AR5L'}">
+      <xacro:include filename="$(find rokae_description)/urdf/AR5-5_07L-W4C4A2.urdf.xacro"/>
+      <xacro:include filename="$(find rokae_description)/urdf/AR5-5_07L-W4C4A2.ros2_control.xacro"/>
+      <xacro:AR5L_ros2_control
+        robot_ip="${robot_ip}"
+        local_ip="${local_ip}"
+        use_fake_hardware="${use_fake_hardware}"/>
+    </xacro:if>
+    <!-- AR5R -->
+    <xacro:if value="${xMate_type == 'AR5R'}">
+      <xacro:include filename="$(find rokae_description)/urdf/AR5-5_07R-W4C4A2.urdf.xacro"/>
+      <xacro:include filename="$(find rokae_description)/urdf/AR5-5_07R-W4C4A2.ros2_control.xacro"/>
+      <xacro:AR5R_ros2_control
+        robot_ip="${robot_ip}"
+        local_ip="${local_ip}"
+        use_fake_hardware="${use_fake_hardware}"/>
+    </xacro:if>
   </xacro:macro>
 </robot>
