Commit message: 适配更多机型

File: rokae/rokae_description/urdf/xMate.urdf.xacro (robot description, xacro)
@@ -30,4 +30,22 @@
     <xacro:property name="xMate_type" value="AR5R"/>
   </xacro:if>
+  <xacro:if value="${robot_type_prop == 'SR5'}">
+    <xacro:property name="xMate_type" value="xMateSR5"/>
+  </xacro:if>
+  <xacro:if value="${robot_type_prop == 'CR12'}">
+    <xacro:property name="xMate_type" value="xMateCR12"/>
+  </xacro:if>
+  <xacro:if value="${robot_type_prop == 'CR18'}">
+    <xacro:property name="xMate_type" value="xMateCR18"/>
+  </xacro:if>
+  <xacro:if value="${robot_type_prop == 'CR20'}">
+    <xacro:property name="xMate_type" value="xMateCR20"/>
+  </xacro:if>
+  <xacro:if value="${robot_type_prop == 'ER3'}">
+    <xacro:property name="xMate_type" value="xMateER3"/>
+  </xacro:if>
+  <xacro:if value="${robot_type_prop == 'SR3'}">
+    <xacro:property name="xMate_type" value="xMateSR3"/>
+  </xacro:if>
   <!-- 调用总宏（只传 xMate_type，内部再按机型 include/调用具体实现） -->
   <xacro:rokae_robot

File: rokae/rokae_description/urdf/xMateER7.ros2_control.xacro (robot description, xacro)
@@ -24,30 +24,30 @@
         </xacro:unless>
       </hardware>
-      <joint name="xMate7_joint_1">
+      <joint name="xMateER7_joint_1">
         <command_interface name="position"/>
         <state_interface name="position"/>
         <state_interface name="velocity"/>
       </joint>
-      <joint name="xMate7_joint_2">
+      <joint name="xMateER7_joint_2">
         <command_interface name="position"/>
         <state_interface name="position"/>
         <state_interface name="velocity"/>
       </joint>
-      <joint name="xMate7_joint_3">
+      <joint name="xMateER7_joint_3">
         <command_interface name="position"/>
         <state_interface name="position"/>
         <state_interface name="velocity"/>
       </joint>
-      <joint name="xMate7_joint_4">
+      <joint name="xMateER7_joint_4">
         <command_interface name="position"/>
         <state_interface name="position"/>
         <state_interface name="velocity"/>
       </joint>
-      <joint name="xMate7_joint_5">
+      <joint name="xMateER7_joint_5">
         <command_interface name="position"/>
         <state_interface name="position"/>
         <state_interface name="velocity"/>
       </joint>
-      <joint name="xMate7_joint_6">
+      <joint name="xMateER7_joint_6">
         <command_interface name="position"/>
         <state_interface name="position"/>

File: rokae/rokae_description/urdf/xMateER7.urdf.xacro (robot description, xacro)
@@ -1,4 +1,4 @@
 <?xml version='1.0' encoding='UTF-8'?>
-<robot xmlns:xacro="http://www.ros.org/wiki/xacro" name="xMate7">
+<robot xmlns:xacro="http://www.ros.org/wiki/xacro" name="xMateER7">
   <!-- Constants for robot dimensions -->
   <!-- <material name="black">
@@ -35,25 +35,25 @@
   <joint name="fixed" type="fixed">
     <parent link="world"/>
-    <child link="xMate7_base"/>
+    <child link="xMateER7_base"/>
   </joint>
   <!--base-->
-  <link name="xMate7_base">
-    <visual>
-      <geometry>
-        <mesh filename="package://rokae_description/meshes/${nameofManipulator}/visual/xMate7_base.stl" scale="0.001 0.001 0.001"/>
-      </geometry>
-      <origin rpy="0 0 0" xyz="0.0 0.0 0.0"/>
-      <material name="white"/>
-    </visual>
-    <collision>
-      <geometry>
-        <mesh filename="package://rokae_description/meshes/${nameofManipulator}/collision/xMate7_base.stl" scale="0.001 0.001 0.001"/>
-      </geometry>
-      <origin rpy="0 0 0" xyz="0.0 0.0 0.0"/>
-    </collision>
-  </link>
-  <joint name="xMate7_joint_1" type="revolute">
-    <parent link="xMate7_base"/>
-    <child link="xMate7_link1"/>
+  <link name="xMateER7_base">
+    <visual>
+      <geometry>
+        <mesh filename="package://rokae_description/meshes/${nameofManipulator}/visual/xMateER7_base.stl" scale="0.001 0.001 0.001"/>
+      </geometry>
+      <origin rpy="0 0 0" xyz="0.0 0.0 0.0"/>
+      <material name="white"/>
+    </visual>
+    <collision>
+      <geometry>
+        <mesh filename="package://rokae_description/meshes/${nameofManipulator}/collision/xMateER7_base.stl" scale="0.001 0.001 0.001"/>
+      </geometry>
+      <origin rpy="0 0 0" xyz="0.0 0.0 0.0"/>
+    </collision>
+  </link>
+  <joint name="xMateER7_joint_1" type="revolute">
+    <parent link="xMateER7_base"/>
+    <child link="xMateER7_link1"/>
     <limit effort="217" lower="-2.9671" upper="2.9671" velocity="1.5707963267948966"/>
     <axis xyz="0 0 1"/>
@@ -62,5 +62,5 @@
   <transmission name="tran1">
     <type>transmission_interface/SimpleTransmission</type>
-    <joint name="xMate7_joint_7">
+    <joint name="xMateER7_joint_7">
       <hardwareInterface>EffortJointInterface</hardwareInterface>
     </joint>
@@ -71,8 +71,8 @@
   </transmission>
   <!--link 1-->
-  <link name="xMate7_link1">
-    <visual>
-      <geometry>
-        <mesh filename="package://rokae_description/meshes/${nameofManipulator}/visual/xMate7_link1.stl" scale="0.001 0.001 0.001"/>
+  <link name="xMateER7_link1">
+    <visual>
+      <geometry>
+        <mesh filename="package://rokae_description/meshes/${nameofManipulator}/visual/xMateER7_link1.stl" scale="0.001 0.001 0.001"/>
       </geometry>
       <origin rpy="0 0 0" xyz="0 0 0"/>
@@ -86,12 +86,12 @@
     <collision>
       <geometry>
-        <mesh filename="package://rokae_description/meshes/${nameofManipulator}/collision/xMate7_link1.stl" scale="0.001 0.001 0.001"/>
-      </geometry>
-      <origin rpy="0 0 0" xyz="0 0 0"/>
-    </collision>
-  </link>
-  <joint name="xMate7_joint_2" type="revolute">
-    <parent link="xMate7_link1"/>
-    <child link="xMate7_link2"/>
+        <mesh filename="package://rokae_description/meshes/${nameofManipulator}/collision/xMateER7_link1.stl" scale="0.001 0.001 0.001"/>
+      </geometry>
+      <origin rpy="0 0 0" xyz="0 0 0"/>
+    </collision>
+  </link>
+  <joint name="xMateER7_joint_2" type="revolute">
+    <parent link="xMateER7_link1"/>
+    <child link="xMateER7_link2"/>
     <limit effort="217" lower="-2.0944" upper="2.0944" velocity="1.5707963267948966"/>
     <axis xyz="0 1 0"/>
@@ -109,8 +109,8 @@
   </transmission>
   <!--link 2-->
-  <link name="xMate7_link2">
-    <visual>
-      <geometry>
-        <mesh filename="package://rokae_description/meshes/${nameofManipulator}/visual/xMate7_link2.stl" scale="0.001 0.001 0.001"/>
+  <link name="xMateER7_link2">
+    <visual>
+      <geometry>
+        <mesh filename="package://rokae_description/meshes/${nameofManipulator}/visual/xMateER7_link2.stl" scale="0.001 0.001 0.001"/>
       </geometry>
       <origin rpy="0 0 0" xyz="0 0 0.0"/>
@@ -124,12 +124,12 @@
     <collision>
       <geometry>
-        <mesh filename="package://rokae_description/meshes/${nameofManipulator}/collision/xMate7_link2.stl" scale="0.001 0.001 0.001"/>
+        <mesh filename="package://rokae_description/meshes/${nameofManipulator}/collision/xMateER7_link2.stl" scale="0.001 0.001 0.001"/>
       </geometry>
       <origin rpy="0 0 0" xyz="0 0 0.0"/>
     </collision>
   </link>
-  <joint name="xMate7_joint_3" type="revolute">
-    <parent link="xMate7_link2"/>
-    <child link="xMate7_link3"/>
+  <joint name="xMateER7_joint_3" type="revolute">
+    <parent link="xMateER7_link2"/>
+    <child link="xMateER7_link3"/>
     <limit effort="102" lower="-2.0944" upper="2.0944" velocity="3.141592653589793"/>
     <axis xyz="0 1 0"/>
@@ -147,8 +147,8 @@
   </transmission>
   <!--link 3-->
-  <link name="xMate7_link3">
-    <visual>
-      <geometry>
-        <mesh filename="package://rokae_description/meshes/${nameofManipulator}/visual/xMate7_link3.stl" scale="0.001 0.001 0.001"/>
+  <link name="xMateER7_link3">
+    <visual>
+      <geometry>
+        <mesh filename="package://rokae_description/meshes/${nameofManipulator}/visual/xMateER7_link3.stl" scale="0.001 0.001 0.001"/>
       </geometry>
       <origin rpy="0 0 0" xyz="0 0 0"/>
@@ -162,12 +162,12 @@
     <collision>
       <geometry>
-        <mesh filename="package://rokae_description/meshes/${nameofManipulator}/collision/xMate7_link3.stl" scale="0.001 0.001 0.001"/>
-      </geometry>
-      <origin rpy="0 0 0" xyz="0 0 0"/>
-    </collision>
-  </link>
-  <joint name="xMate7_joint_4" type="revolute">
-    <parent link="xMate7_link3"/>
-    <child link="xMate7_link4"/>
+        <mesh filename="package://rokae_description/meshes/${nameofManipulator}/collision/xMateER7_link3.stl" scale="0.001 0.001 0.001"/>
+      </geometry>
+      <origin rpy="0 0 0" xyz="0 0 0"/>
+    </collision>
+  </link>
+  <joint name="xMateER7_joint_4" type="revolute">
+    <parent link="xMateER7_link3"/>
+    <child link="xMateER7_link4"/>
     <limit effort="66" lower="-2.9671" upper="2.9671" velocity="3.141592653589793"/>
     <!--     lower="-6.2832" upper="6.2832" -->
@@ -187,8 +187,8 @@
   </transmission>
   <!--link 4-->
-  <link name="xMate7_link4">
-    <visual>
-      <geometry>
-        <mesh filename="package://rokae_description/meshes/${nameofManipulator}/visual/xMate7_link4.stl" scale=".001 0.001 0.001"/>
+  <link name="xMateER7_link4">
+    <visual>
+      <geometry>
+        <mesh filename="package://rokae_description/meshes/${nameofManipulator}/visual/xMateER7_link4.stl" scale=".001 0.001 0.001"/>
       </geometry>
       <origin rpy="0 0 0" xyz="0.0 0.0 0.0"/>
@@ -202,12 +202,12 @@
     <collision>
       <geometry>
-        <mesh filename="package://rokae_description/meshes/${nameofManipulator}/collision/xMate7_link4.stl" scale="0.001 0.001 0.001"/>
-      </geometry>
-      <origin rpy="0 0 0" xyz="0.0 0.0 0.0"/>
-    </collision>
-  </link>
-  <joint name="xMate7_joint_5" type="revolute">
-    <parent link="xMate7_link4"/>
-    <child link="xMate7_link5"/>
+        <mesh filename="package://rokae_description/meshes/${nameofManipulator}/collision/xMateER7_link4.stl" scale="0.001 0.001 0.001"/>
+      </geometry>
+      <origin rpy="0 0 0" xyz="0.0 0.0 0.0"/>
+    </collision>
+  </link>
+  <joint name="xMateER7_joint_5" type="revolute">
+    <parent link="xMateER7_link4"/>
+    <child link="xMateER7_link5"/>
     <limit effort="66" lower="-2.0944" upper="2.0944" velocity="3.141592653589793"/>
     <axis xyz="0 1 0"/>
@@ -225,8 +225,8 @@
   </transmission>
   <!--link 5-->
-  <link name="xMate7_link5">
-    <visual>
-      <geometry>
-        <mesh filename="package://rokae_description/meshes/${nameofManipulator}/visual/xMate7_link5.stl" scale="0.001 0.001 0.001"/>
+  <link name="xMateER7_link5">
+    <visual>
+      <geometry>
+        <mesh filename="package://rokae_description/meshes/${nameofManipulator}/visual/xMateER7_link5.stl" scale="0.001 0.001 0.001"/>
       </geometry>
       <origin rpy="0 0 0" xyz="0 0 0"/>
@@ -240,12 +240,12 @@
     <collision>
       <geometry>
-        <mesh filename="package://rokae_description/meshes/${nameofManipulator}/collision/xMate7_link5.stl" scale="0.001 0.001 0.001"/>
-      </geometry>
-      <origin rpy="0 0 0" xyz="0 0 0"/>
-    </collision>
-  </link>
-  <joint name="xMate7_joint_6" type="revolute">
-    <parent link="xMate7_link5"/>
-    <child link="xMate7_link6"/>
+        <mesh filename="package://rokae_description/meshes/${nameofManipulator}/collision/xMateER7_link5.stl" scale="0.001 0.001 0.001"/>
+      </geometry>
+      <origin rpy="0 0 0" xyz="0 0 0"/>
+    </collision>
+  </link>
+  <joint name="xMateER7_joint_6" type="revolute">
+    <parent link="xMateER7_link5"/>
+    <child link="xMateER7_link6"/>
     <limit effort="66" lower="-6.2832" upper="6.2832" velocity="3.141592653589793"/>
     <axis xyz="0 0 1"/>
@@ -263,8 +263,8 @@
   </transmission>
   <!--link 6-->
-  <link name="xMate7_link6">
-    <visual>
-      <geometry>
-        <mesh filename="package://rokae_description/meshes/${nameofManipulator}/visual/xMate7_link6.stl" scale="0.001 0.001 0.001"/>
+  <link name="xMateER7_link6">
+    <visual>
+      <geometry>
+        <mesh filename="package://rokae_description/meshes/${nameofManipulator}/visual/xMateER7_link6.stl" scale="0.001 0.001 0.001"/>
       </geometry>
       <origin rpy="0 0 0" xyz="0.0 0.0 0.0"/>
@@ -278,5 +278,5 @@
     <collision>
       <geometry>
-        <mesh filename="package://rokae_description/meshes/${nameofManipulator}/collision/xMate7_link6.stl" scale="0.001 0.001 0.001"/>
+        <mesh filename="package://rokae_description/meshes/${nameofManipulator}/collision/xMateER7_link6.stl" scale="0.001 0.001 0.001"/>
       </geometry>
       <origin rpy="0 0 0" xyz="0.0 0.0 0.0"/>

File: rokae/rokae_description/urdf/xMatePro3.urdf.xacro (robot description, xacro)
@@ -39,5 +39,5 @@
     <parent link="${nameofManipulator}_base"/>
     <child link="${nameofManipulator}_link1"/>
- <limit effort="300" lower="-3.0527" upper="3.0527" velocity="10"/>
+ <limit effort="300" lower="-3.0527" upper="3.0527" velocity="3"/>
     <axis xyz="0 0 1"/>
     <origin rpy="0 0 0" xyz="0 0 0"/>
@@ -77,5 +77,5 @@
     <parent link="${nameofManipulator}_link1"/>
     <child link="${nameofManipulator}_link2"/>
-  <limit effort="300" lower="-2.0933" upper="2.0933" velocity="10"/>
+  <limit effort="300" lower="-2.0933" upper="2.0933" velocity="3"/>
     <axis xyz="0 1 0"/>
 	<origin rpy="0 0 0" xyz="0 0 0.34260487"/>
@@ -115,5 +115,5 @@
     <parent link="${nameofManipulator}_link2"/>
     <child link="${nameofManipulator}_link3"/>
-  <limit effort="300" lower="-3.0527" upper="3.0527" velocity="10"/>
+  <limit effort="300" lower="-3.0527" upper="3.0527" velocity="3"/>
     <axis xyz="0 0 1"/>
     <origin rpy="0 0 0" xyz="0 0 0.23743878"/>
@@ -153,5 +153,5 @@
     <parent link="${nameofManipulator}_link3"/>
     <child link="${nameofManipulator}_link4"/>
-   <limit effort="300" lower="-2.0933" upper="2.0933" velocity="10"/>
+   <limit effort="300" lower="-2.0933" upper="2.0933" velocity="3"/>
 <!--     lower="-2.79" upper="2.79" -->
     <axis xyz="0 1 0"/>
@@ -193,5 +193,5 @@
     <parent link="${nameofManipulator}_link4"/>
     <child link="${nameofManipulator}_link5"/>
-  <limit effort="300" lower="-3.0527" upper="3.0527" velocity="10"/>
+  <limit effort="300" lower="-3.0527" upper="3.0527" velocity="3"/>
     <axis xyz="0 0 1"/>
    <origin rpy="0 0 0" xyz="0 0 0.22044633"/>
@@ -231,5 +231,5 @@
     <parent link="${nameofManipulator}_link5"/>
     <child link="${nameofManipulator}_link6"/>
-   <limit effort="300" lower="-2.0933" upper="2.0933" velocity="10"/>
+   <limit effort="300" lower="-2.0933" upper="2.0933" velocity="3"/>
     <axis xyz="0 1 0"/>
     <origin rpy="0.0 0.0 0" xyz="0 0 0.14512568" />
@@ -269,5 +269,5 @@
     <parent link="${nameofManipulator}_link6"/>
     <child link="${nameofManipulator}_link7"/>
-   <limit effort="300" lower="-6.283" upper="6.283" velocity="10"/>
+   <limit effort="300" lower="-6.283" upper="6.283" velocity="3"/>
     <axis xyz="0 0 1"/>
     <origin rpy="0.0 0.0 0.0" xyz="0 0 0.25090877" />

File: rokae/rokae_description/urdf/xMatePro7.urdf.xacro (robot description, xacro)
@@ -39,5 +39,5 @@
     <parent link="${nameofManipulator}_base"/>
     <child link="${nameofManipulator}_link1"/>
- <limit effort="300" lower="-3.0527" upper="3.0527" velocity="10"/>
+ <limit effort="300" lower="-3.0527" upper="3.0527" velocity="3"/>
     <axis xyz="0 0 1"/>
     <origin rpy="0 0 0" xyz="0 0 0"/>
@@ -77,5 +77,5 @@
     <parent link="${nameofManipulator}_link1"/>
     <child link="${nameofManipulator}_link2"/>
-  <limit effort="300" lower="-2.0933" upper="2.0933" velocity="10"/>
+  <limit effort="300" lower="-2.0933" upper="2.0933" velocity="3"/>
     <axis xyz="0 1 0"/>
 	<origin rpy="0 0 0" xyz="0 0 0.404"/>
@@ -115,5 +115,5 @@
     <parent link="${nameofManipulator}_link2"/>
     <child link="${nameofManipulator}_link3"/>
-  <limit effort="300" lower="-3.0527" upper="3.0527" velocity="10"/>
+  <limit effort="300" lower="-3.0527" upper="3.0527" velocity="3"/>
     <axis xyz="0 0 1"/>
     <origin rpy="0 0 0" xyz="0 0 0.23743878"/>
@@ -153,5 +153,5 @@
     <parent link="${nameofManipulator}_link3"/>
     <child link="${nameofManipulator}_link4"/>
-   <limit effort="300" lower="-2.0933" upper="2.0933" velocity="10"/>
+   <limit effort="300" lower="-2.0933" upper="2.0933" velocity="3"/>
 <!--     lower="-2.79" upper="2.79" -->
     <axis xyz="0 1 0"/>
@@ -193,5 +193,5 @@
     <parent link="${nameofManipulator}_link4"/>
     <child link="${nameofManipulator}_link5"/>
-  <limit effort="300" lower="-3.0527" upper="3.0527" velocity="10"/>
+  <limit effort="300" lower="-3.0527" upper="3.0527" velocity="3"/>
     <axis xyz="0 0 1"/>
    <origin rpy="0 0 0" xyz="0 0 0.22044633"/>
@@ -231,5 +231,5 @@
     <parent link="${nameofManipulator}_link5"/>
     <child link="${nameofManipulator}_link6"/>
-   <limit effort="300" lower="-2.0933" upper="2.0933" velocity="10"/>
+   <limit effort="300" lower="-2.0933" upper="2.0933" velocity="3"/>
     <axis xyz="0 1 0"/>
     <origin rpy="0.0 0.0 0" xyz="0 0 0.14512568" />
@@ -269,5 +269,5 @@
     <parent link="${nameofManipulator}_link6"/>
     <child link="${nameofManipulator}_link7"/>
-   <limit effort="300" lower="-6.283" upper="6.283" velocity="10"/>
+   <limit effort="300" lower="-6.283" upper="6.283" velocity="3"/>
     <axis xyz="0 0 1"/>
     <origin rpy="0.0 0.0 0.0" xyz="0 0 0.25090877" />

File: rokae/rokae_description/urdf/xMate_macro.xacro (robot description, xacro)
@@ -53,5 +53,4 @@
         use_fake_hardware="${use_fake_hardware}"/>
     </xacro:if>
-    <!-- 其他机型（如有）按同样模式继续加 -->
     <!-- AR5L -->
     <xacro:if value="${xMate_type == 'AR5L'}">
@@ -72,4 +71,53 @@
         use_fake_hardware="${use_fake_hardware}"/>
     </xacro:if>
+    <xacro:if value="${xMate_type == 'xMateSR5'}">
+      <xacro:include filename="$(find rokae_description)/urdf/xMateSR5.urdf.xacro"/>
+      <xacro:include filename="$(find rokae_description)/urdf/xMateSR5.ros2_control.xacro"/>
+      <xacro:sr5_ros2_control
+        robot_ip="${robot_ip}"
+        local_ip="${local_ip}"
+        use_fake_hardware="${use_fake_hardware}"/>
+    </xacro:if>
+    <xacro:if value="${xMate_type == 'xMateCR12'}">
+      <xacro:include filename="$(find rokae_description)/urdf/xMateCR12.urdf.xacro"/>
+      <xacro:include filename="$(find rokae_description)/urdf/xMateCR12.ros2_control.xacro"/>
+      <xacro:cr12_ros2_control
+        robot_ip="${robot_ip}"
+        local_ip="${local_ip}"
+        use_fake_hardware="${use_fake_hardware}"/>
+    </xacro:if>
+    <xacro:if value="${xMate_type == 'xMateCR18'}">
+      <xacro:include filename="$(find rokae_description)/urdf/xMateCR18.urdf.xacro"/>
+      <xacro:include filename="$(find rokae_description)/urdf/xMateCR18.ros2_control.xacro"/>
+      <xacro:cr18_ros2_control
+        robot_ip="${robot_ip}"
+        local_ip="${local_ip}"
+        use_fake_hardware="${use_fake_hardware}"/>
+    </xacro:if>
+    <xacro:if value="${xMate_type == 'xMateCR20'}">
+      <xacro:include filename="$(find rokae_description)/urdf/xMateCR20.urdf.xacro"/>
+      <xacro:include filename="$(find rokae_description)/urdf/xMateCR20.ros2_control.xacro"/>
+      <xacro:cr20_ros2_control
+        robot_ip="${robot_ip}"
+        local_ip="${local_ip}"
+        use_fake_hardware="${use_fake_hardware}"/>
+    </xacro:if>
+    <xacro:if value="${xMate_type == 'xMateER3'}">
+      <xacro:include filename="$(find rokae_description)/urdf/xMateER3.urdf.xacro"/>
+      <xacro:include filename="$(find rokae_description)/urdf/xMateER3.ros2_control.xacro"/>
+      <xacro:er3_ros2_control
+        robot_ip="${robot_ip}"
+        local_ip="${local_ip}"
+        use_fake_hardware="${use_fake_hardware}"/>
+    </xacro:if>
+    <xacro:if value="${xMate_type == 'xMateSR3'}">
+      <xacro:include filename="$(find rokae_description)/urdf/xMateSR3.urdf.xacro"/>
+      <xacro:include filename="$(find rokae_description)/urdf/xMateSR3.ros2_control.xacro"/>
+      <xacro:sr3_ros2_control
+        robot_ip="${robot_ip}"
+        local_ip="${local_ip}"
+        use_fake_hardware="${use_fake_hardware}"/>
+    </xacro:if>
+    <!-- 其他机型（如有）按同样模式继续加 -->
   </xacro:macro>
 </robot>
