Commit message: 更新

File: rokae_description/urdf/xMateCR7.urdf.xacro (robot description, xacro)
@@ -39,5 +39,5 @@
     <parent link="${nameofManipulator}_base"/>
     <child link="${nameofManipulator}_link1"/>
- <limit effort="300" lower="-3.054" upper="3.054" velocity="8"/>
+ <limit effort="194" lower="-3.0543" upper="3.0543" velocity="3.141592653589793"/>
     <axis xyz="0 0 1"/>
     <origin rpy="0 0 0" xyz="0 0 0"/>
@@ -77,5 +77,5 @@
     <parent link="${nameofManipulator}_link1"/>
     <child link="${nameofManipulator}_link2"/>
-  <limit effort="300" lower="-3.054" upper="3.054" velocity="8"/>
+  <limit effort="194" lower="-3.0543" upper="3.0543" velocity="3.141592653589793"/>
     <axis xyz="0 1 0"/>
 	<origin rpy="0 0 0" xyz="0 0 0.296"/>
@@ -115,5 +115,5 @@
     <parent link="${nameofManipulator}_link2"/>
     <child link="${nameofManipulator}_link3"/>
-  <limit effort="300" lower="-3.054" upper="3.054" velocity="8"/>
+  <limit effort="102" lower="-3.0543" upper="3.0543" velocity="4.084070449666731"/>
     <axis xyz="0 -1 0"/>
     <origin rpy="0 0 0" xyz="0 0 0.49"/>
@@ -153,5 +153,5 @@
     <parent link="${nameofManipulator}_link3"/>
     <child link="${nameofManipulator}_link4"/>
-   <limit effort="300" lower="-3.054" upper="3.054" velocity="8"/>
+   <limit effort="66" lower="-3.0543" upper="3.0543" velocity="4.1887902047863905"/>
 <!--     lower="-2.79" upper="2.79" -->
     <axis xyz="0 0 1"/>
@@ -193,5 +193,5 @@
     <parent link="${nameofManipulator}_link4"/>
     <child link="${nameofManipulator}_link5"/>
-  <limit effort="300" lower="-3.054" upper="3.054" velocity="8"/>
+  <limit effort="66" lower="-3.0543" upper="3.0543" velocity="4.1887902047863905"/>
     <axis xyz="0 -1 0"/>
    <origin rpy="0 0 0" xyz="0 -0.151 0"/>
@@ -231,5 +231,5 @@
     <parent link="${nameofManipulator}_link5"/>
     <child link="${nameofManipulator}_link6"/>
-   <limit effort="300" lower="-3.054" upper="3.054" velocity="8"/>
+   <limit effort="29" lower="-3.0543" upper="3.0543" velocity="5.235987755982989"/>
     <axis xyz="0 0 1"/>
     <origin rpy="0.0 0.0 0" xyz="0 0 0.1265" />

File: rokae_description/urdf/xMatePro3.urdf.xacro (robot description, xacro)
@@ -39,5 +39,5 @@
     <parent link="${nameofManipulator}_base"/>
     <child link="${nameofManipulator}_link1"/>
- <limit effort="300" lower="-3.0527" upper="3.0527" velocity="3"/>
+ <limit effort="102" lower="-2.9671" upper="2.9671" velocity="3.141592653589793"/>
     <axis xyz="0 0 1"/>
     <origin rpy="0 0 0" xyz="0 0 0"/>
@@ -77,5 +77,5 @@
     <parent link="${nameofManipulator}_link1"/>
     <child link="${nameofManipulator}_link2"/>
-  <limit effort="300" lower="-2.0933" upper="2.0933" velocity="3"/>
+  <limit effort="108" lower="-2.0944" upper="2.0944" velocity="2.6179938779914944"/>
     <axis xyz="0 1 0"/>
 	<origin rpy="0 0 0" xyz="0 0 0.34260487"/>
@@ -115,5 +115,5 @@
     <parent link="${nameofManipulator}_link2"/>
     <child link="${nameofManipulator}_link3"/>
-  <limit effort="300" lower="-3.0527" upper="3.0527" velocity="3"/>
+  <limit effort="102" lower="-2.9671" upper="2.9671" velocity="3.141592653589793"/>
     <axis xyz="0 0 1"/>
     <origin rpy="0 0 0" xyz="0 0 0.23743878"/>
@@ -153,5 +153,5 @@
     <parent link="${nameofManipulator}_link3"/>
     <child link="${nameofManipulator}_link4"/>
-   <limit effort="300" lower="-2.0933" upper="2.0933" velocity="3"/>
+   <limit effort="102" lower="-2.0944" upper="2.0944" velocity="3.141592653589793"/>
 <!--     lower="-2.79" upper="2.79" -->
     <axis xyz="0 1 0"/>
@@ -193,5 +193,5 @@
     <parent link="${nameofManipulator}_link4"/>
     <child link="${nameofManipulator}_link5"/>
-  <limit effort="300" lower="-3.0527" upper="3.0527" velocity="3"/>
+  <limit effort="29" lower="-2.9671" upper="2.9671" velocity="3.9269908169872414"/>
     <axis xyz="0 0 1"/>
    <origin rpy="0 0 0" xyz="0 0 0.22044633"/>
@@ -231,5 +231,5 @@
     <parent link="${nameofManipulator}_link5"/>
     <child link="${nameofManipulator}_link6"/>
-   <limit effort="300" lower="-2.0933" upper="2.0933" velocity="3"/>
+   <limit effort="29" lower="-2.0944" upper="2.0944" velocity="3.9269908169872414"/>
     <axis xyz="0 1 0"/>
     <origin rpy="0.0 0.0 0" xyz="0 0 0.14512568" />
@@ -269,5 +269,5 @@
     <parent link="${nameofManipulator}_link6"/>
     <child link="${nameofManipulator}_link7"/>
-   <limit effort="300" lower="-6.283" upper="6.283" velocity="3"/>
+   <limit effort="29" lower="-6.2832" upper="6.2832" velocity="3.9269908169872414"/>
     <axis xyz="0 0 1"/>
     <origin rpy="0.0 0.0 0.0" xyz="0 0 0.25090877" />

File: rokae_description/urdf/xMatePro7.urdf.xacro (robot description, xacro)
@@ -39,5 +39,5 @@
     <parent link="${nameofManipulator}_base"/>
     <child link="${nameofManipulator}_link1"/>
- <limit effort="300" lower="-3.0527" upper="3.0527" velocity="3"/>
+ <limit effort="217" lower="-2.9671" upper="2.9671" velocity="1.5707963267948966"/>
     <axis xyz="0 0 1"/>
     <origin rpy="0 0 0" xyz="0 0 0"/>
@@ -77,5 +77,5 @@
     <parent link="${nameofManipulator}_link1"/>
     <child link="${nameofManipulator}_link2"/>
-  <limit effort="300" lower="-2.0933" upper="2.0933" velocity="3"/>
+  <limit effort="217" lower="-2.0944" upper="2.0944" velocity="1.5707963267948966"/>
     <axis xyz="0 1 0"/>
 	<origin rpy="0 0 0" xyz="0 0 0.404"/>
@@ -115,5 +115,5 @@
     <parent link="${nameofManipulator}_link2"/>
     <child link="${nameofManipulator}_link3"/>
-  <limit effort="300" lower="-3.0527" upper="3.0527" velocity="3"/>
+  <limit effort="102" lower="-2.9671" upper="2.9671" velocity="2.0943951023931953"/>
     <axis xyz="0 0 1"/>
     <origin rpy="0 0 0" xyz="0 0 0.23743878"/>
@@ -153,5 +153,5 @@
     <parent link="${nameofManipulator}_link3"/>
     <child link="${nameofManipulator}_link4"/>
-   <limit effort="300" lower="-2.0933" upper="2.0933" velocity="3"/>
+   <limit effort="102" lower="-2.0944" upper="2.0944" velocity="2.0943951023931953"/>
 <!--     lower="-2.79" upper="2.79" -->
     <axis xyz="0 1 0"/>
@@ -193,5 +193,5 @@
     <parent link="${nameofManipulator}_link4"/>
     <child link="${nameofManipulator}_link5"/>
-  <limit effort="300" lower="-3.0527" upper="3.0527" velocity="3"/>
+  <limit effort="66" lower="-2.9671" upper="2.9671" velocity="2.0943951023931953"/>
     <axis xyz="0 0 1"/>
    <origin rpy="0 0 0" xyz="0 0 0.22044633"/>
@@ -231,5 +231,5 @@
     <parent link="${nameofManipulator}_link5"/>
     <child link="${nameofManipulator}_link6"/>
-   <limit effort="300" lower="-2.0933" upper="2.0933" velocity="3"/>
+   <limit effort="66" lower="-2.0944" upper="2.0944" velocity="2.0943951023931953"/>
     <axis xyz="0 1 0"/>
     <origin rpy="0.0 0.0 0" xyz="0 0 0.14512568" />
@@ -269,5 +269,5 @@
     <parent link="${nameofManipulator}_link6"/>
     <child link="${nameofManipulator}_link7"/>
-   <limit effort="300" lower="-6.283" upper="6.283" velocity="3"/>
+   <limit effort="66" lower="-6.2832" upper="6.2832" velocity="2.0943951023931953"/>
     <axis xyz="0 0 1"/>
     <origin rpy="0.0 0.0 0.0" xyz="0 0 0.25090877" />

File: rokae_description/urdf/xMateSR4.urdf.xacro (robot description, xacro)
@@ -39,5 +39,5 @@
     <parent link="${nameofManipulator}_base"/>
     <child link="${nameofManipulator}_link1"/>
- <limit effort="300" lower="-3.1416" upper="3.1416" velocity="10"/>
+ <limit effort="102" lower="-3.0543" upper="3.0543" velocity="3.141592653589793"/>
     <axis xyz="0 0 1"/>
     <origin rpy="0 0 0" xyz="0 0 0"/>
@@ -77,5 +77,5 @@
     <parent link="${nameofManipulator}_link1"/>
     <child link="${nameofManipulator}_link2"/>
-  <limit effort="300" lower="-2.4222" upper="2.35619" velocity="10"/>
+  <limit effort="102" lower="-2.3562" upper="2.3562" velocity="3.141592653589793"/>
     <axis xyz="0 1 0"/>
 	<origin rpy="0 0 0" xyz="0 0 0.355"/>
@@ -115,5 +115,5 @@
     <parent link="${nameofManipulator}_link2"/>
     <child link="${nameofManipulator}_link3"/>
-  <limit effort="300" lower="-2.96555" upper="2.35619" velocity="10"/>
+  <limit effort="102" lower="-2.3562" upper="2.3562" velocity="3.141592653589793"/>
     <axis xyz="0 -1 0"/>
     <origin rpy="0 0 0" xyz="0.05 0 0.4"/>
@@ -153,5 +153,5 @@
     <parent link="${nameofManipulator}_link3"/>
     <child link="${nameofManipulator}_link4"/>
-   <limit effort="300" lower="-3.1416" upper="3.1416" velocity="10"/>
+   <limit effort="16" lower="-3.0543" upper="3.0543" velocity="3.141592653589793"/>
 <!--     lower="-2.79" upper="2.79" -->
     <axis xyz="0 0 1"/>
@@ -193,5 +193,5 @@
     <parent link="${nameofManipulator}_link4"/>
     <child link="${nameofManipulator}_link5"/>
-  <limit effort="300" lower="-3.1416" upper="3.1416" velocity="10"/>
+  <limit effort="16" lower="-3.0543" upper="3.0543" velocity="3.141592653589793"/>
     <axis xyz="0 -1 0"/>
    <origin rpy="0 0 0" xyz="0 0.136 0"/>
@@ -231,5 +231,5 @@
     <parent link="${nameofManipulator}_link5"/>
     <child link="${nameofManipulator}_link6"/>
-   <limit effort="300" lower="-3.14" upper="3.14" velocity="10"/>
+   <limit effort="16" lower="-3.0543" upper="3.0543" velocity="3.141592653589793"/>
     <axis xyz="0 0 1"/>
     <origin rpy="0.0 0.0 0" xyz="0 0 0.1035" />
