Commit message: 适配CR35机型

File: rokae_description/urdf/xMate.urdf.xacro (robot description, xacro)
@@ -2,5 +2,5 @@
 <robot xmlns:xacro="http://www.ros.org/wiki/xacro" name="xMate_robot">
   <!-- 启动参数（launch.py 会传 robot_type） -->
-  <xacro:arg name="robot_type" default="CR7"/>  <!-- 可选: CR7, SR4, ER7p, ER7 -->
+  <xacro:arg name="robot_type" default="CR7"/>  <!-- 可选: CR7, CR12, CR18, CR20, CR35, SR4, ... -->
   <xacro:arg name="robot_ip" default="192.168.21.10"/>
   <xacro:arg name="local_ip" default="192.168.21.131"/>
@@ -42,4 +42,7 @@
     <xacro:property name="xMate_type" value="xMateCR20"/>
   </xacro:if>
+  <xacro:if value="${robot_type_prop == 'CR35'}">
+    <xacro:property name="xMate_type" value="xMateCR35"/>
+  </xacro:if>
   <xacro:if value="${robot_type_prop == 'ER3'}">
     <xacro:property name="xMate_type" value="xMateER3"/>

File: rokae_description/urdf/xMate_macro.xacro (robot description, xacro)
@@ -103,4 +103,12 @@
         use_fake_hardware="${use_fake_hardware}"/>
     </xacro:if>
+    <xacro:if value="${xMate_type == 'xMateCR35'}">
+      <xacro:include filename="$(find rokae_description)/urdf/xMateCR35.urdf.xacro"/>
+      <xacro:include filename="$(find rokae_description)/urdf/xMateCR35.ros2_control.xacro"/>
+      <xacro:cr35_ros2_control
+        robot_ip="${robot_ip}"
+        local_ip="${local_ip}"
+        use_fake_hardware="${use_fake_hardware}"/>
+    </xacro:if>
     <xacro:if value="${xMate_type == 'xMateER3'}">
       <xacro:include filename="$(find rokae_description)/urdf/xMateER3.urdf.xacro"/>
