Commit message: 添加gazebo功能

File: rokae_description/urdf/AR5-5_07L-W4C4A2.ros2_control.xacro (robot description, xacro)
@@ -24,35 +24,35 @@
         </xacro:unless>
       </hardware>
-      <joint name="AR5-5_07L-W4C4A2_joint_1">
+      <joint name="joint1">
         <command_interface name="position"/>
         <state_interface name="position"/>
         <state_interface name="velocity"/>
       </joint>
-      <joint name="AR5-5_07L-W4C4A2_joint_2">
+      <joint name="joint2">
         <command_interface name="position"/>
         <state_interface name="position"/>
         <state_interface name="velocity"/>
       </joint>
-      <joint name="AR5-5_07L-W4C4A2_joint_3">
+      <joint name="joint3">
         <command_interface name="position"/>
         <state_interface name="position"/>
         <state_interface name="velocity"/>
       </joint>
-      <joint name="AR5-5_07L-W4C4A2_joint_4">
+      <joint name="joint4">
         <command_interface name="position"/>
         <state_interface name="position"/>
         <state_interface name="velocity"/>
       </joint>
-      <joint name="AR5-5_07L-W4C4A2_joint_5">
+      <joint name="joint5">
         <command_interface name="position"/>
         <state_interface name="position"/>
         <state_interface name="velocity"/>
       </joint>
-      <joint name="AR5-5_07L-W4C4A2_joint_6">
+      <joint name="joint6">
         <command_interface name="position"/>
         <state_interface name="position"/>
         <state_interface name="velocity"/>
       </joint>
-      <joint name="AR5-5_07L-W4C4A2_joint_7">
+      <joint name="joint7">
         <command_interface name="position"/>
         <state_interface name="position"/>

File: rokae_description/urdf/AR5-5_07L-W4C4A2.urdf.xacro (robot description, xacro)
@@ -27,5 +27,5 @@
     </collision>
   </link>
-  <joint name="AR5-5_07L-W4C4A2_joint_1" type="revolute">
+  <joint name="joint1" type="revolute">
     <parent link="AR5-5_07L-W4C4A2_base"/>
     <child link="AR5-5_07L-W4C4A2_link1"/>
@@ -36,5 +36,5 @@
   <transmission name="tran1">
     <type>transmission_interface/SimpleTransmission</type>
-    <joint name="AR5-5_07L-W4C4A2_joint_8">
+    <joint name="joint1">
       <hardwareInterface>EffortJointInterface</hardwareInterface>
     </joint>
@@ -65,5 +65,5 @@
     </collision>
   </link>
-  <joint name="AR5-5_07L-W4C4A2_joint_2" type="revolute">
+  <joint name="joint2" type="revolute">
     <parent link="AR5-5_07L-W4C4A2_link1"/>
     <child link="AR5-5_07L-W4C4A2_link2"/>
@@ -74,5 +74,5 @@
   <transmission name="tran2">
     <type>transmission_interface/SimpleTransmission</type>
-    <joint name="xmate_joint_2">
+    <joint name="joint2">
       <hardwareInterface>EffortJointInterface</hardwareInterface>
     </joint>
@@ -103,5 +103,5 @@
     </collision>
   </link>
-  <joint name="AR5-5_07L-W4C4A2_joint_3" type="revolute">
+  <joint name="joint3" type="revolute">
     <parent link="AR5-5_07L-W4C4A2_link2"/>
     <child link="AR5-5_07L-W4C4A2_link3"/>
@@ -112,5 +112,5 @@
   <transmission name="tran3">
     <type>transmission_interface/SimpleTransmission</type>
-    <joint name="xmate_joint_3">
+    <joint name="joint3">
       <hardwareInterface>EffortJointInterface</hardwareInterface>
     </joint>
@@ -141,5 +141,5 @@
     </collision>
   </link>
-  <joint name="AR5-5_07L-W4C4A2_joint_4" type="revolute">
+  <joint name="joint4" type="revolute">
     <parent link="AR5-5_07L-W4C4A2_link3"/>
     <child link="AR5-5_07L-W4C4A2_link4"/>
@@ -152,5 +152,5 @@
   <transmission name="tran4">
     <type>transmission_interface/SimpleTransmission</type>
-    <joint name="xmate_joint_4">
+    <joint name="joint4">
       <hardwareInterface>EffortJointInterface</hardwareInterface>
     </joint>
@@ -181,5 +181,5 @@
     </collision>
   </link>
-  <joint name="AR5-5_07L-W4C4A2_joint_5" type="revolute">
+  <joint name="joint5" type="revolute">
     <parent link="AR5-5_07L-W4C4A2_link4"/>
     <child link="AR5-5_07L-W4C4A2_link5"/>
@@ -190,5 +190,5 @@
   <transmission name="tran5">
     <type>transmission_interface/SimpleTransmission</type>
-    <joint name="xmate_joint_5">
+    <joint name="joint5">
       <hardwareInterface>EffortJointInterface</hardwareInterface>
     </joint>
@@ -219,5 +219,5 @@
     </collision>
   </link>
-  <joint name="AR5-5_07L-W4C4A2_joint_6" type="revolute">
+  <joint name="joint6" type="revolute">
     <parent link="AR5-5_07L-W4C4A2_link5"/>
     <child link="AR5-5_07L-W4C4A2_link6"/>
@@ -228,5 +228,5 @@
   <transmission name="tran6">
     <type>transmission_interface/SimpleTransmission</type>
-    <joint name="xmate_joint_6">
+    <joint name="joint6">
       <hardwareInterface>EffortJointInterface</hardwareInterface>
     </joint>
@@ -257,5 +257,5 @@
     </collision>
   </link>
-  <joint name="AR5-5_07L-W4C4A2_joint_7" type="revolute">
+  <joint name="joint7" type="revolute">
     <parent link="AR5-5_07L-W4C4A2_link6"/>
     <child link="AR5-5_07L-W4C4A2_link7"/>

File: rokae_description/urdf/AR5-5_07R-W4C4A2.ros2_control.xacro (robot description, xacro)
@@ -24,35 +24,35 @@
         </xacro:unless>
       </hardware>
-      <joint name="AR5-5_07R-W4C4A2_joint_1">
+      <joint name="joint1">
         <command_interface name="position"/>
         <state_interface name="position"/>
         <state_interface name="velocity"/>
       </joint>
-      <joint name="AR5-5_07R-W4C4A2_joint_2">
+      <joint name="joint2">
         <command_interface name="position"/>
         <state_interface name="position"/>
         <state_interface name="velocity"/>
       </joint>
-      <joint name="AR5-5_07R-W4C4A2_joint_3">
+      <joint name="joint3">
         <command_interface name="position"/>
         <state_interface name="position"/>
         <state_interface name="velocity"/>
       </joint>
-      <joint name="AR5-5_07R-W4C4A2_joint_4">
+      <joint name="joint4">
         <command_interface name="position"/>
         <state_interface name="position"/>
         <state_interface name="velocity"/>
       </joint>
-      <joint name="AR5-5_07R-W4C4A2_joint_5">
+      <joint name="joint5">
         <command_interface name="position"/>
         <state_interface name="position"/>
         <state_interface name="velocity"/>
       </joint>
-      <joint name="AR5-5_07R-W4C4A2_joint_6">
+      <joint name="joint6">
         <command_interface name="position"/>
         <state_interface name="position"/>
         <state_interface name="velocity"/>
       </joint>
-      <joint name="AR5-5_07R-W4C4A2_joint_7">
+      <joint name="joint7">
         <command_interface name="position"/>
         <state_interface name="position"/>

File: rokae_description/urdf/AR5-5_07R-W4C4A2.urdf.xacro (robot description, xacro)
@@ -52,5 +52,5 @@
     </collision>
   </link>
-  <joint name="AR5-5_07R-W4C4A2_joint_1" type="revolute">
+  <joint name="joint1" type="revolute">
     <parent link="AR5-5_07R-W4C4A2_base"/>
     <child link="AR5-5_07R-W4C4A2_link1"/>
@@ -61,5 +61,5 @@
   <transmission name="tran1">
     <type>transmission_interface/SimpleTransmission</type>
-    <joint name="AR5-5_07R-W4C4A2_joint_8">
+    <joint name="joint1">
       <hardwareInterface>EffortJointInterface</hardwareInterface>
     </joint>
@@ -90,5 +90,5 @@
     </collision>
   </link>
-  <joint name="AR5-5_07R-W4C4A2_joint_2" type="revolute">
+  <joint name="joint2" type="revolute">
     <parent link="AR5-5_07R-W4C4A2_link1"/>
     <child link="AR5-5_07R-W4C4A2_link2"/>
@@ -99,5 +99,5 @@
   <transmission name="tran2">
     <type>transmission_interface/SimpleTransmission</type>
-    <joint name="xmate_joint_2">
+    <joint name="joint2">
       <hardwareInterface>EffortJointInterface</hardwareInterface>
     </joint>
@@ -128,5 +128,5 @@
     </collision>
   </link>
-  <joint name="AR5-5_07R-W4C4A2_joint_3" type="revolute">
+  <joint name="joint3" type="revolute">
     <parent link="AR5-5_07R-W4C4A2_link2"/>
     <child link="AR5-5_07R-W4C4A2_link3"/>
@@ -137,5 +137,5 @@
   <transmission name="tran3">
     <type>transmission_interface/SimpleTransmission</type>
-    <joint name="xmate_joint_3">
+    <joint name="joint3">
       <hardwareInterface>EffortJointInterface</hardwareInterface>
     </joint>
@@ -166,5 +166,5 @@
     </collision>
   </link>
-  <joint name="AR5-5_07R-W4C4A2_joint_4" type="revolute">
+  <joint name="joint4" type="revolute">
     <parent link="AR5-5_07R-W4C4A2_link3"/>
     <child link="AR5-5_07R-W4C4A2_link4"/>
@@ -177,5 +177,5 @@
   <transmission name="tran4">
     <type>transmission_interface/SimpleTransmission</type>
-    <joint name="xmate_joint_4">
+    <joint name="joint4">
       <hardwareInterface>EffortJointInterface</hardwareInterface>
     </joint>
@@ -206,5 +206,5 @@
     </collision>
   </link>
-  <joint name="AR5-5_07R-W4C4A2_joint_5" type="revolute">
+  <joint name="joint5" type="revolute">
     <parent link="AR5-5_07R-W4C4A2_link4"/>
     <child link="AR5-5_07R-W4C4A2_link5"/>
@@ -215,5 +215,5 @@
   <transmission name="tran5">
     <type>transmission_interface/SimpleTransmission</type>
-    <joint name="xmate_joint_5">
+    <joint name="joint5">
       <hardwareInterface>EffortJointInterface</hardwareInterface>
     </joint>
@@ -244,5 +244,5 @@
     </collision>
   </link>
-  <joint name="AR5-5_07R-W4C4A2_joint_6" type="revolute">
+  <joint name="joint6" type="revolute">
     <parent link="AR5-5_07R-W4C4A2_link5"/>
     <child link="AR5-5_07R-W4C4A2_link6"/>
@@ -253,5 +253,5 @@
   <transmission name="tran6">
     <type>transmission_interface/SimpleTransmission</type>
-    <joint name="xmate_joint_6">
+    <joint name="joint6">
       <hardwareInterface>EffortJointInterface</hardwareInterface>
     </joint>
@@ -282,5 +282,5 @@
     </collision>
   </link>
-  <joint name="AR5-5_07R-W4C4A2_joint_7" type="revolute">
+  <joint name="joint7" type="revolute">
     <parent link="AR5-5_07R-W4C4A2_link6"/>
     <child link="AR5-5_07R-W4C4A2_link7"/>

File: rokae_description/urdf/xMateCR12.ros2_control.xacro (robot description, xacro)
@@ -24,30 +24,30 @@
         </xacro:unless>
       </hardware>
-      <joint name="xMateCR12_joint_1">
+      <joint name="joint1">
         <command_interface name="position"/>
         <state_interface name="position"/>
         <state_interface name="velocity"/>
       </joint>
-      <joint name="xMateCR12_joint_2">
+      <joint name="joint2">
         <command_interface name="position"/>
         <state_interface name="position"/>
         <state_interface name="velocity"/>
       </joint>
-      <joint name="xMateCR12_joint_3">
+      <joint name="joint3">
         <command_interface name="position"/>
         <state_interface name="position"/>
         <state_interface name="velocity"/>
       </joint>
-      <joint name="xMateCR12_joint_4">
+      <joint name="joint4">
         <command_interface name="position"/>
         <state_interface name="position"/>
         <state_interface name="velocity"/>
       </joint>
-      <joint name="xMateCR12_joint_5">
+      <joint name="joint5">
         <command_interface name="position"/>
         <state_interface name="position"/>
         <state_interface name="velocity"/>
       </joint>
-      <joint name="xMateCR12_joint_6">
+      <joint name="joint6">
         <command_interface name="position"/>
         <state_interface name="position"/>

File: rokae_description/urdf/xMateCR12.urdf.xacro (robot description, xacro)
@@ -51,5 +51,5 @@
     </collision>
   </link>
-  <joint name="xMateCR12_joint_1" type="revolute">
+  <joint name="joint1" type="revolute">
     <parent link="xMateCR12_base"/>
     <child link="xMateCR12_link1"/>
@@ -89,5 +89,5 @@
     </collision>
   </link>
-  <joint name="xMateCR12_joint_2" type="revolute">
+  <joint name="joint2" type="revolute">
     <parent link="xMateCR12_link1"/>
     <child link="xMateCR12_link2"/>
@@ -98,5 +98,5 @@
   <transmission name="tran2">
     <type>transmission_interface/SimpleTransmission</type>
-    <joint name="xmate_joint_2">
+    <joint name="joint2">
       <hardwareInterface>EffortJointInterface</hardwareInterface>
     </joint>
@@ -127,5 +127,5 @@
     </collision>
   </link>
-  <joint name="xMateCR12_joint_3" type="revolute">
+  <joint name="joint3" type="revolute">
     <parent link="xMateCR12_link2"/>
     <child link="xMateCR12_link3"/>
@@ -136,5 +136,5 @@
   <transmission name="tran3">
     <type>transmission_interface/SimpleTransmission</type>
-    <joint name="xmate_joint_3">
+    <joint name="joint3">
       <hardwareInterface>EffortJointInterface</hardwareInterface>
     </joint>
@@ -165,5 +165,5 @@
     </collision>
   </link>
-  <joint name="xMateCR12_joint_4" type="revolute">
+  <joint name="joint4" type="revolute">
     <parent link="xMateCR12_link3"/>
     <child link="xMateCR12_link4"/>
@@ -176,5 +176,5 @@
   <transmission name="tran4">
     <type>transmission_interface/SimpleTransmission</type>
-    <joint name="xmate_joint_4">
+    <joint name="joint4">
       <hardwareInterface>EffortJointInterface</hardwareInterface>
     </joint>
@@ -205,5 +205,5 @@
     </collision>
   </link>
-  <joint name="xMateCR12_joint_5" type="revolute">
+  <joint name="joint5" type="revolute">
     <parent link="xMateCR12_link4"/>
     <child link="xMateCR12_link5"/>
@@ -214,5 +214,5 @@
   <transmission name="tran5">
     <type>transmission_interface/SimpleTransmission</type>
-    <joint name="xmate_joint_5">
+    <joint name="joint5">
       <hardwareInterface>EffortJointInterface</hardwareInterface>
     </joint>
@@ -243,5 +243,5 @@
     </collision>
   </link>
-  <joint name="xMateCR12_joint_6" type="revolute">
+  <joint name="joint6" type="revolute">
     <parent link="xMateCR12_link5"/>
     <child link="xMateCR12_link6"/>
@@ -252,5 +252,5 @@
   <transmission name="tran6">
     <type>transmission_interface/SimpleTransmission</type>
-    <joint name="xmate_joint_6">
+    <joint name="joint6">
       <hardwareInterface>EffortJointInterface</hardwareInterface>
     </joint>

File: rokae_description/urdf/xMateCR18.ros2_control.xacro (robot description, xacro)
@@ -24,30 +24,30 @@
         </xacro:unless>
       </hardware>
-      <joint name="xMateCR18_joint_1">
+      <joint name="joint1">
         <command_interface name="position"/>
         <state_interface name="position"/>
         <state_interface name="velocity"/>
       </joint>
-      <joint name="xMateCR18_joint_2">
+      <joint name="joint2">
         <command_interface name="position"/>
         <state_interface name="position"/>
         <state_interface name="velocity"/>
       </joint>
-      <joint name="xMateCR18_joint_3">
+      <joint name="joint3">
         <command_interface name="position"/>
         <state_interface name="position"/>
         <state_interface name="velocity"/>
       </joint>
-      <joint name="xMateCR18_joint_4">
+      <joint name="joint4">
         <command_interface name="position"/>
         <state_interface name="position"/>
         <state_interface name="velocity"/>
       </joint>
-      <joint name="xMateCR18_joint_5">
+      <joint name="joint5">
         <command_interface name="position"/>
         <state_interface name="position"/>
         <state_interface name="velocity"/>
       </joint>
-      <joint name="xMateCR18_joint_6">
+      <joint name="joint6">
         <command_interface name="position"/>
         <state_interface name="position"/>

File: rokae_description/urdf/xMateCR18.urdf.xacro (robot description, xacro)
@@ -51,5 +51,5 @@
     </collision>
   </link>
-  <joint name="xMateCR18_joint_1" type="revolute">
+  <joint name="joint1" type="revolute">
     <parent link="xMateCR18_base"/>
     <child link="xMateCR18_link1"/>
@@ -89,5 +89,5 @@
     </collision>
   </link>
-  <joint name="xMateCR18_joint_2" type="revolute">
+  <joint name="joint2" type="revolute">
     <parent link="xMateCR18_link1"/>
     <child link="xMateCR18_link2"/>
@@ -98,5 +98,5 @@
   <transmission name="tran2">
     <type>transmission_interface/SimpleTransmission</type>
-    <joint name="xmate_joint_2">
+    <joint name="joint2">
       <hardwareInterface>EffortJointInterface</hardwareInterface>
     </joint>
@@ -127,5 +127,5 @@
     </collision>
   </link>
-  <joint name="xMateCR18_joint_3" type="revolute">
+  <joint name="joint3" type="revolute">
     <parent link="xMateCR18_link2"/>
     <child link="xMateCR18_link3"/>
@@ -136,5 +136,5 @@
   <transmission name="tran3">
     <type>transmission_interface/SimpleTransmission</type>
-    <joint name="xmate_joint_3">
+    <joint name="joint3">
       <hardwareInterface>EffortJointInterface</hardwareInterface>
     </joint>
@@ -165,5 +165,5 @@
     </collision>
   </link>
-  <joint name="xMateCR18_joint_4" type="revolute">
+  <joint name="joint4" type="revolute">
     <parent link="xMateCR18_link3"/>
     <child link="xMateCR18_link4"/>
@@ -176,5 +176,5 @@
   <transmission name="tran4">
     <type>transmission_interface/SimpleTransmission</type>
-    <joint name="xmate_joint_4">
+    <joint name="joint4">
       <hardwareInterface>EffortJointInterface</hardwareInterface>
     </joint>
@@ -205,5 +205,5 @@
     </collision>
   </link>
-  <joint name="xMateCR18_joint_5" type="revolute">
+  <joint name="joint5" type="revolute">
     <parent link="xMateCR18_link4"/>
     <child link="xMateCR18_link5"/>
@@ -214,5 +214,5 @@
   <transmission name="tran5">
     <type>transmission_interface/SimpleTransmission</type>
-    <joint name="xmate_joint_5">
+    <joint name="joint5">
       <hardwareInterface>EffortJointInterface</hardwareInterface>
     </joint>
@@ -243,5 +243,5 @@
     </collision>
   </link>
-  <joint name="xMateCR18_joint_6" type="revolute">
+  <joint name="joint6" type="revolute">
     <parent link="xMateCR18_link5"/>
     <child link="xMateCR18_link6"/>
@@ -252,5 +252,5 @@
   <transmission name="tran6">
     <type>transmission_interface/SimpleTransmission</type>
-    <joint name="xmate_joint_6">
+    <joint name="joint6">
       <hardwareInterface>EffortJointInterface</hardwareInterface>
     </joint>

File: rokae_description/urdf/xMateCR20.ros2_control.xacro (robot description, xacro)
@@ -24,30 +24,30 @@
         </xacro:unless>
       </hardware>
-      <joint name="xMateCR20_joint_1">
+      <joint name="joint1">
         <command_interface name="position"/>
         <state_interface name="position"/>
         <state_interface name="velocity"/>
       </joint>
-      <joint name="xMateCR20_joint_2">
+      <joint name="joint2">
         <command_interface name="position"/>
         <state_interface name="position"/>
         <state_interface name="velocity"/>
       </joint>
-      <joint name="xMateCR20_joint_3">
+      <joint name="joint3">
         <command_interface name="position"/>
         <state_interface name="position"/>
         <state_interface name="velocity"/>
       </joint>
-      <joint name="xMateCR20_joint_4">
+      <joint name="joint4">
         <command_interface name="position"/>
         <state_interface name="position"/>
         <state_interface name="velocity"/>
       </joint>
-      <joint name="xMateCR20_joint_5">
+      <joint name="joint5">
         <command_interface name="position"/>
         <state_interface name="position"/>
         <state_interface name="velocity"/>
       </joint>
-      <joint name="xMateCR20_joint_6">
+      <joint name="joint6">
         <command_interface name="position"/>
         <state_interface name="position"/>

File: rokae_description/urdf/xMateCR20.urdf.xacro (robot description, xacro)
@@ -51,5 +51,5 @@
     </collision>
   </link>
-  <joint name="xMateCR20_joint_1" type="revolute">
+  <joint name="joint1" type="revolute">
     <parent link="xMateCR20_base"/>
     <child link="xMateCR20_link1"/>
@@ -89,5 +89,5 @@
     </collision>
   </link>
-  <joint name="xMateCR20_joint_2" type="revolute">
+  <joint name="joint2" type="revolute">
     <parent link="xMateCR20_link1"/>
     <child link="xMateCR20_link2"/>
@@ -98,5 +98,5 @@
   <transmission name="tran2">
     <type>transmission_interface/SimpleTransmission</type>
-    <joint name="xmate_joint_2">
+    <joint name="joint2">
       <hardwareInterface>EffortJointInterface</hardwareInterface>
     </joint>
@@ -127,5 +127,5 @@
     </collision>
   </link>
-  <joint name="xMateCR20_joint_3" type="revolute">
+  <joint name="joint3" type="revolute">
     <parent link="xMateCR20_link2"/>
     <child link="xMateCR20_link3"/>
@@ -136,5 +136,5 @@
   <transmission name="tran3">
     <type>transmission_interface/SimpleTransmission</type>
-    <joint name="xmate_joint_3">
+    <joint name="joint3">
       <hardwareInterface>EffortJointInterface</hardwareInterface>
     </joint>
@@ -165,5 +165,5 @@
     </collision>
   </link>
-  <joint name="xMateCR20_joint_4" type="revolute">
+  <joint name="joint4" type="revolute">
     <parent link="xMateCR20_link3"/>
     <child link="xMateCR20_link4"/>
@@ -176,5 +176,5 @@
   <transmission name="tran4">
     <type>transmission_interface/SimpleTransmission</type>
-    <joint name="xmate_joint_4">
+    <joint name="joint4">
       <hardwareInterface>EffortJointInterface</hardwareInterface>
     </joint>
@@ -205,5 +205,5 @@
     </collision>
   </link>
-  <joint name="xMateCR20_joint_5" type="revolute">
+  <joint name="joint5" type="revolute">
     <parent link="xMateCR20_link4"/>
     <child link="xMateCR20_link5"/>
@@ -214,5 +214,5 @@
   <transmission name="tran5">
     <type>transmission_interface/SimpleTransmission</type>
-    <joint name="xmate_joint_5">
+    <joint name="joint5">
       <hardwareInterface>EffortJointInterface</hardwareInterface>
     </joint>
@@ -243,5 +243,5 @@
     </collision>
   </link>
-  <joint name="xMateCR20_joint_6" type="revolute">
+  <joint name="joint6" type="revolute">
     <parent link="xMateCR20_link5"/>
     <child link="xMateCR20_link6"/>
@@ -252,5 +252,5 @@
   <transmission name="tran6">
     <type>transmission_interface/SimpleTransmission</type>
-    <joint name="xmate_joint_6">
+    <joint name="joint6">
       <hardwareInterface>EffortJointInterface</hardwareInterface>
     </joint>

File: rokae_description/urdf/xMateCR7.ros2_control.xacro (robot description, xacro)
@@ -22,4 +22,7 @@
           <param name="local_ip">${local_ip}</param>
           <param name="xMate_type">${xMate_type}</param>
+          <!-- 与 controller_manager 实际更新周期一致（常见 250Hz→0.004）；仅 enable_servoj=true 时才会调用 setServoJoint -->
+          <param name="servo_joint_period_s">0.004</param>
+          <param name="enable_servoj">false</param>
         </xacro:unless>
       </hardware>

File: rokae_description/urdf/xMateCR7.urdf.xacro (robot description, xacro)
@@ -3,4 +3,7 @@
 <!--  Attention!!! inertia in the model is not correct!!! -->
 <robot name="xMateCR7" xmlns:xacro="http://www.ros.org/wiki/xacro">
+  <!-- Real hardware: passed from launch (xacro mappings) -->
+  <xacro:arg name="robot_ip" default="10.0.2.163"/>
+  <xacro:arg name="local_ip" default="10.0.2.162"/>
   <!-- Constants for robot dimensions -->
   <!-- Import all Gazebo-customization elements, including Gazebo colors -->
