Commit message: 添加gazebo功能

File: rokae_description/urdf/xMateER3.ros2_control.xacro (robot description, xacro)
@@ -24,30 +24,30 @@
         </xacro:unless>
       </hardware>
-      <joint name="xMateER3_joint_1">
+      <joint name="joint1">
         <command_interface name="position"/>
         <state_interface name="position"/>
         <state_interface name="velocity"/>
       </joint>
-      <joint name="xMateER3_joint_2">
+      <joint name="joint2">
         <command_interface name="position"/>
         <state_interface name="position"/>
         <state_interface name="velocity"/>
       </joint>
-      <joint name="xMateER3_joint_3">
+      <joint name="joint3">
         <command_interface name="position"/>
         <state_interface name="position"/>
         <state_interface name="velocity"/>
       </joint>
-      <joint name="xMateER3_joint_4">
+      <joint name="joint4">
         <command_interface name="position"/>
         <state_interface name="position"/>
         <state_interface name="velocity"/>
       </joint>
-      <joint name="xMateER3_joint_5">
+      <joint name="joint5">
         <command_interface name="position"/>
         <state_interface name="position"/>
         <state_interface name="velocity"/>
       </joint>
-      <joint name="xMateER3_joint_6">
+      <joint name="joint6">
         <command_interface name="position"/>
         <state_interface name="position"/>

File: rokae_description/urdf/xMateER3.urdf.xacro (robot description, xacro)
@@ -51,5 +51,5 @@
     </collision>
   </link>
-  <joint name="xMateER3_joint_1" type="revolute">
+  <joint name="joint1" type="revolute">
     <parent link="xMateER3_base"/>
     <child link="xMateER3_link1"/>
@@ -60,5 +60,5 @@
   <transmission name="tran1">
     <type>transmission_interface/SimpleTransmission</type>
-    <joint name="xMateER3_joint_7">
+    <joint name="joint1">
       <hardwareInterface>EffortJointInterface</hardwareInterface>
     </joint>
@@ -89,5 +89,5 @@
     </collision>
   </link>
-  <joint name="xMateER3_joint_2" type="revolute">
+  <joint name="joint2" type="revolute">
     <parent link="xMateER3_link1"/>
     <child link="xMateER3_link2"/>
@@ -98,5 +98,5 @@
   <transmission name="tran2">
     <type>transmission_interface/SimpleTransmission</type>
-    <joint name="xmate_joint_2">
+    <joint name="joint2">
       <hardwareInterface>EffortJointInterface</hardwareInterface>
     </joint>
@@ -127,5 +127,5 @@
     </collision>
   </link>
-  <joint name="xMateER3_joint_3" type="revolute">
+  <joint name="joint3" type="revolute">
     <parent link="xMateER3_link2"/>
     <child link="xMateER3_link3"/>
@@ -136,5 +136,5 @@
   <transmission name="tran3">
     <type>transmission_interface/SimpleTransmission</type>
-    <joint name="xmate_joint_3">
+    <joint name="joint3">
       <hardwareInterface>EffortJointInterface</hardwareInterface>
     </joint>
@@ -165,5 +165,5 @@
     </collision>
   </link>
-  <joint name="xMateER3_joint_4" type="revolute">
+  <joint name="joint4" type="revolute">
     <parent link="xMateER3_link3"/>
     <child link="xMateER3_link4"/>
@@ -176,5 +176,5 @@
   <transmission name="tran4">
     <type>transmission_interface/SimpleTransmission</type>
-    <joint name="xmate_joint_4">
+    <joint name="joint4">
       <hardwareInterface>EffortJointInterface</hardwareInterface>
     </joint>
@@ -205,5 +205,5 @@
     </collision>
   </link>
-  <joint name="xMateER3_joint_5" type="revolute">
+  <joint name="joint5" type="revolute">
     <parent link="xMateER3_link4"/>
     <child link="xMateER3_link5"/>
@@ -214,5 +214,5 @@
   <transmission name="tran5">
     <type>transmission_interface/SimpleTransmission</type>
-    <joint name="xmate_joint_5">
+    <joint name="joint5">
       <hardwareInterface>EffortJointInterface</hardwareInterface>
     </joint>
@@ -243,5 +243,5 @@
     </collision>
   </link>
-  <joint name="xMateER3_joint_6" type="revolute">
+  <joint name="joint6" type="revolute">
     <parent link="xMateER3_link5"/>
     <child link="xMateER3_link6"/>
@@ -252,5 +252,5 @@
   <transmission name="tran6">
     <type>transmission_interface/SimpleTransmission</type>
-    <joint name="xmate_joint_6">
+    <joint name="joint6">
       <hardwareInterface>EffortJointInterface</hardwareInterface>
     </joint>

File: rokae_description/urdf/xMateER7.ros2_control.xacro (robot description, xacro)
@@ -24,30 +24,30 @@
         </xacro:unless>
       </hardware>
-      <joint name="xMateER7_joint_1">
+      <joint name="joint1">
         <command_interface name="position"/>
         <state_interface name="position"/>
         <state_interface name="velocity"/>
       </joint>
-      <joint name="xMateER7_joint_2">
+      <joint name="joint2">
         <command_interface name="position"/>
         <state_interface name="position"/>
         <state_interface name="velocity"/>
       </joint>
-      <joint name="xMateER7_joint_3">
+      <joint name="joint3">
         <command_interface name="position"/>
         <state_interface name="position"/>
         <state_interface name="velocity"/>
       </joint>
-      <joint name="xMateER7_joint_4">
+      <joint name="joint4">
         <command_interface name="position"/>
         <state_interface name="position"/>
         <state_interface name="velocity"/>
       </joint>
-      <joint name="xMateER7_joint_5">
+      <joint name="joint5">
         <command_interface name="position"/>
         <state_interface name="position"/>
         <state_interface name="velocity"/>
       </joint>
-      <joint name="xMateER7_joint_6">
+      <joint name="joint6">
         <command_interface name="position"/>
         <state_interface name="position"/>

File: rokae_description/urdf/xMateER7.urdf.xacro (robot description, xacro)
@@ -53,5 +53,5 @@
     </collision>
   </link>
-  <joint name="xMateER7_joint_1" type="revolute">
+  <joint name="joint1" type="revolute">
     <parent link="xMateER7_base"/>
     <child link="xMateER7_link1"/>
@@ -91,5 +91,5 @@
     </collision>
   </link>
-  <joint name="xMateER7_joint_2" type="revolute">
+  <joint name="joint2" type="revolute">
     <parent link="xMateER7_link1"/>
     <child link="xMateER7_link2"/>
@@ -100,5 +100,5 @@
   <transmission name="tran2">
     <type>transmission_interface/SimpleTransmission</type>
-    <joint name="xmate_joint_2">
+    <joint name="joint2">
       <hardwareInterface>EffortJointInterface</hardwareInterface>
     </joint>
@@ -129,5 +129,5 @@
     </collision>
   </link>
-  <joint name="xMateER7_joint_3" type="revolute">
+  <joint name="joint3" type="revolute">
     <parent link="xMateER7_link2"/>
     <child link="xMateER7_link3"/>
@@ -138,5 +138,5 @@
   <transmission name="tran3">
     <type>transmission_interface/SimpleTransmission</type>
-    <joint name="xmate_joint_3">
+    <joint name="joint3">
       <hardwareInterface>EffortJointInterface</hardwareInterface>
     </joint>
@@ -167,5 +167,5 @@
     </collision>
   </link>
-  <joint name="xMateER7_joint_4" type="revolute">
+  <joint name="joint4" type="revolute">
     <parent link="xMateER7_link3"/>
     <child link="xMateER7_link4"/>
@@ -178,5 +178,5 @@
   <transmission name="tran4">
     <type>transmission_interface/SimpleTransmission</type>
-    <joint name="xmate_joint_4">
+    <joint name="joint4">
       <hardwareInterface>EffortJointInterface</hardwareInterface>
     </joint>
@@ -207,5 +207,5 @@
     </collision>
   </link>
-  <joint name="xMateER7_joint_5" type="revolute">
+  <joint name="joint5" type="revolute">
     <parent link="xMateER7_link4"/>
     <child link="xMateER7_link5"/>
@@ -216,5 +216,5 @@
   <transmission name="tran5">
     <type>transmission_interface/SimpleTransmission</type>
-    <joint name="xmate_joint_5">
+    <joint name="joint5">
       <hardwareInterface>EffortJointInterface</hardwareInterface>
     </joint>
@@ -245,5 +245,5 @@
     </collision>
   </link>
-  <joint name="xMateER7_joint_6" type="revolute">
+  <joint name="joint6" type="revolute">
     <parent link="xMateER7_link5"/>
     <child link="xMateER7_link6"/>
@@ -254,5 +254,5 @@
   <transmission name="tran6">
     <type>transmission_interface/SimpleTransmission</type>
-    <joint name="xmate_joint_6">
+    <joint name="joint6">
       <hardwareInterface>EffortJointInterface</hardwareInterface>
     </joint>

File: rokae_description/urdf/xMatePro3.urdf.xacro (robot description, xacro)
@@ -45,5 +45,5 @@
 <transmission name="tran1">
     <type>transmission_interface/SimpleTransmission</type>
-    <joint name="xmate_joint_1">
+    <joint name="joint1">
       <hardwareInterface>EffortJointInterface</hardwareInterface>
     </joint>
@@ -83,5 +83,5 @@
    <transmission name="tran2">
      <type>transmission_interface/SimpleTransmission</type>
-    <joint name="xmate_joint_2">
+    <joint name="joint2">
       <hardwareInterface>EffortJointInterface</hardwareInterface>
     </joint>
@@ -121,5 +121,5 @@
    <transmission name="tran3">
     <type>transmission_interface/SimpleTransmission</type>
-    <joint name="xmate_joint_3">
+    <joint name="joint3">
       <hardwareInterface>EffortJointInterface</hardwareInterface>
     </joint>
@@ -161,5 +161,5 @@
   <transmission name="tran4">
     <type>transmission_interface/SimpleTransmission</type>
-    <joint name="xmate_joint_4">
+    <joint name="joint4">
       <hardwareInterface>EffortJointInterface</hardwareInterface>
     </joint>
@@ -199,5 +199,5 @@
   <transmission name="tran5">
     <type>transmission_interface/SimpleTransmission</type>
-    <joint name="xmate_joint_5">
+    <joint name="joint5">
       <hardwareInterface>EffortJointInterface</hardwareInterface>
     </joint>
@@ -237,5 +237,5 @@
   <transmission name="tran6">
     <type>transmission_interface/SimpleTransmission</type>
-    <joint name="xmate_joint_6">
+    <joint name="joint6">
       <hardwareInterface>EffortJointInterface</hardwareInterface>
     </joint>

File: rokae_description/urdf/xMatePro7.urdf.xacro (robot description, xacro)
@@ -45,5 +45,5 @@
 <transmission name="tran1">
     <type>transmission_interface/SimpleTransmission</type>
-    <joint name="xmate_joint_1">
+    <joint name="joint1">
       <hardwareInterface>EffortJointInterface</hardwareInterface>
     </joint>
@@ -83,5 +83,5 @@
    <transmission name="tran2">
      <type>transmission_interface/SimpleTransmission</type>
-    <joint name="xmate_joint_2">
+    <joint name="joint2">
       <hardwareInterface>EffortJointInterface</hardwareInterface>
     </joint>
@@ -121,5 +121,5 @@
    <transmission name="tran3">
     <type>transmission_interface/SimpleTransmission</type>
-    <joint name="xmate_joint_3">
+    <joint name="joint3">
       <hardwareInterface>EffortJointInterface</hardwareInterface>
     </joint>
@@ -161,5 +161,5 @@
   <transmission name="tran4">
     <type>transmission_interface/SimpleTransmission</type>
-    <joint name="xmate_joint_4">
+    <joint name="joint4">
       <hardwareInterface>EffortJointInterface</hardwareInterface>
     </joint>
@@ -199,5 +199,5 @@
   <transmission name="tran5">
     <type>transmission_interface/SimpleTransmission</type>
-    <joint name="xmate_joint_5">
+    <joint name="joint5">
       <hardwareInterface>EffortJointInterface</hardwareInterface>
     </joint>
@@ -237,5 +237,5 @@
   <transmission name="tran6">
     <type>transmission_interface/SimpleTransmission</type>
-    <joint name="xmate_joint_6">
+    <joint name="joint6">
       <hardwareInterface>EffortJointInterface</hardwareInterface>
     </joint>

File: rokae_description/urdf/xMateSR3.ros2_control.xacro (robot description, xacro)
@@ -24,30 +24,30 @@
         </xacro:unless>
       </hardware>
-      <joint name="xMateSR3_joint_1">
+      <joint name="joint1">
         <command_interface name="position"/>
         <state_interface name="position"/>
         <state_interface name="velocity"/>
       </joint>
-      <joint name="xMateSR3_joint_2">
+      <joint name="joint2">
         <command_interface name="position"/>
         <state_interface name="position"/>
         <state_interface name="velocity"/>
       </joint>
-      <joint name="xMateSR3_joint_3">
+      <joint name="joint3">
         <command_interface name="position"/>
         <state_interface name="position"/>
         <state_interface name="velocity"/>
       </joint>
-      <joint name="xMateSR3_joint_4">
+      <joint name="joint4">
         <command_interface name="position"/>
         <state_interface name="position"/>
         <state_interface name="velocity"/>
       </joint>
-      <joint name="xMateSR3_joint_5">
+      <joint name="joint5">
         <command_interface name="position"/>
         <state_interface name="position"/>
         <state_interface name="velocity"/>
       </joint>
-      <joint name="xMateSR3_joint_6">
+      <joint name="joint6">
         <command_interface name="position"/>
         <state_interface name="position"/>

File: rokae_description/urdf/xMateSR3.urdf.xacro (robot description, xacro)
@@ -51,5 +51,5 @@
     </collision>
   </link>
-  <joint name="xMateSR3_joint_1" type="revolute">
+  <joint name="joint1" type="revolute">
     <parent link="xMateSR3_base"/>
     <child link="xMateSR3_link1"/>
@@ -60,5 +60,5 @@
   <transmission name="tran1">
     <type>transmission_interface/SimpleTransmission</type>
-    <joint name="xMateSR3_joint_7">
+    <joint name="joint1">
       <hardwareInterface>EffortJointInterface</hardwareInterface>
     </joint>
@@ -89,5 +89,5 @@
     </collision>
   </link>
-  <joint name="xMateSR3_joint_2" type="revolute">
+  <joint name="joint2" type="revolute">
     <parent link="xMateSR3_link1"/>
     <child link="xMateSR3_link2"/>
@@ -98,5 +98,5 @@
   <transmission name="tran2">
     <type>transmission_interface/SimpleTransmission</type>
-    <joint name="xmate_joint_2">
+    <joint name="joint2">
       <hardwareInterface>EffortJointInterface</hardwareInterface>
     </joint>
@@ -127,5 +127,5 @@
     </collision>
   </link>
-  <joint name="xMateSR3_joint_3" type="revolute">
+  <joint name="joint3" type="revolute">
     <parent link="xMateSR3_link2"/>
     <child link="xMateSR3_link3"/>
@@ -136,5 +136,5 @@
   <transmission name="tran3">
     <type>transmission_interface/SimpleTransmission</type>
-    <joint name="xmate_joint_3">
+    <joint name="joint3">
       <hardwareInterface>EffortJointInterface</hardwareInterface>
     </joint>
@@ -165,5 +165,5 @@
     </collision>
   </link>
-  <joint name="xMateSR3_joint_4" type="revolute">
+  <joint name="joint4" type="revolute">
     <parent link="xMateSR3_link3"/>
     <child link="xMateSR3_link4"/>
@@ -176,5 +176,5 @@
   <transmission name="tran4">
     <type>transmission_interface/SimpleTransmission</type>
-    <joint name="xmate_joint_4">
+    <joint name="joint4">
       <hardwareInterface>EffortJointInterface</hardwareInterface>
     </joint>
@@ -205,5 +205,5 @@
     </collision>
   </link>
-  <joint name="xMateSR3_joint_5" type="revolute">
+  <joint name="joint5" type="revolute">
     <parent link="xMateSR3_link4"/>
     <child link="xMateSR3_link5"/>
@@ -214,5 +214,5 @@
   <transmission name="tran5">
     <type>transmission_interface/SimpleTransmission</type>
-    <joint name="xmate_joint_5">
+    <joint name="joint5">
       <hardwareInterface>EffortJointInterface</hardwareInterface>
     </joint>
@@ -243,5 +243,5 @@
     </collision>
   </link>
-  <joint name="xMateSR3_joint_6" type="revolute">
+  <joint name="joint6" type="revolute">
     <parent link="xMateSR3_link5"/>
     <child link="xMateSR3_link6"/>
@@ -252,5 +252,5 @@
   <transmission name="tran6">
     <type>transmission_interface/SimpleTransmission</type>
-    <joint name="xmate_joint_6">
+    <joint name="joint6">
       <hardwareInterface>EffortJointInterface</hardwareInterface>
     </joint>
